Commit message: Added both kinect transforms ; updated bash scripts to launch everything

File: meka_description/urdf/H2R4_r_hand_defs.urdf.xacro (robot description, xacro)
@@ -132,6 +132,14 @@
       </collision>
     </link>
+    <joint name="right_hand_j3" type="revolute">
+      <axis xyz="0 -1 0" />
+      <origin xyz="-0.035 0 0" rpy="0 0 0" />
+      <parent link="thumb2" />
+      <child link="thumb_end"/>
+      <limit effort="100" velocity="${50*M_PI/180}" lower="${-14.94*M_PI/180}" upper="${14.94*M_PI/180}" />
+    </joint>
+    <link name="thumb_end"/>
 <!-- Start Index Finger -->
-    <joint name="right_hand_j3" type="revolute">
+    <joint name="right_hand_j4" type="revolute">
       <axis xyz="0 1 0" />
       <origin xyz="0 0.028 -0.101" rpy="0 0 0" />
@@ -165,5 +173,5 @@
       </collision>
     </link>
-    <joint name="right_hand_j4" type="revolute">
+    <joint name="right_hand_j5" type="revolute">
       <axis xyz="0 1 0" />
       <limit effort="100" velocity="${1600*M_PI/180}" lower="${-34.99*M_PI/180}" upper="${34.99*M_PI/180}" />
@@ -197,5 +205,5 @@
       </collision>
     </link>
-    <joint name="right_hand_j5" type="revolute">
+    <joint name="right_hand_j6" type="revolute">
       <axis xyz="0 1 0" />
       <limit effort="100" velocity="${1600*M_PI/180}" lower="${-34.21*M_PI/180}" upper="${34.213*M_PI/180}" />
@@ -229,6 +237,14 @@
       </collision>
     </link>
+    <joint name="right_hand_j7" type="revolute">
+      <axis xyz="0 1 0" />
+      <limit effort="100" velocity="${1600*M_PI/180}" lower="${-34.21*M_PI/180}" upper="${34.213*M_PI/180}" />
+      <origin xyz="0 0 -0.025" rpy="0 0 0" />
+      <parent link="index2"/>
+      <child link="index_end"/>
+    </joint>
+    <link name="index_end"/>
 <!-- Start Ring Finger -->
-    <joint name="right_hand_j6" type="revolute">
+    <joint name="right_hand_j8" type="revolute">
       <axis xyz="0 1 0" />
       <origin xyz="0 0 -0.101" rpy="0 0 0" />
@@ -262,5 +278,5 @@
       </collision>
     </link>
-    <joint name="right_hand_j7" type="revolute">
+    <joint name="right_hand_j9" type="revolute">
       <axis xyz="0 1 0" />
       <limit effort="100" velocity="${1600*M_PI/180}" lower="${-34.99*M_PI/180}" upper="${34.99*M_PI/180}" />
@@ -294,5 +310,5 @@
       </collision>
     </link>
-    <joint name="right_hand_j8" type="revolute">
+    <joint name="right_hand_j10" type="revolute">
       <axis xyz="0 1 0" />
       <limit effort="100" velocity="${1600*M_PI/180}" lower="${-34.21*M_PI/180}" upper="${34.213*M_PI/180}" />
@@ -326,6 +342,14 @@
       </collision>
     </link>
+    <joint name="right_hand_j11" type="revolute">
+      <axis xyz="0 1 0" />
+      <limit effort="100" velocity="${1600*M_PI/180}" lower="${-34.21*M_PI/180}" upper="${34.213*M_PI/180}" />
+      <origin xyz="0 0 -0.025" rpy="0 0 0" />
+      <parent link="ring2"/>
+      <child link="ring_end"/>
+    </joint>
+    <link name="ring_end"/>
 <!-- Start Pinky Finger -->
-    <joint name="right_hand_j9" type="revolute">
+    <joint name="right_hand_j12" type="revolute">
       <axis xyz="0 1 0" />
       <origin xyz="0 -0.028 -0.101" rpy="0 0 0" />
@@ -359,5 +383,5 @@
       </collision>
     </link>
-    <joint name="right_hand_j10" type="revolute">
+    <joint name="right_hand_j13" type="revolute">
       <axis xyz="0 1 0" />
       <limit effort="100" velocity="${1600*M_PI/180}" lower="${-34.99*M_PI/180}" upper="${34.99*M_PI/180}" />
@@ -391,5 +415,5 @@
       </collision>
     </link>
-    <joint name="right_hand_j11" type="revolute">
+    <joint name="right_hand_j14" type="revolute">
       <axis xyz="0 1 0" />
       <limit effort="100" velocity="${1600*M_PI/180}" lower="${-34.21*M_PI/180}" upper="${34.213*M_PI/180}" />
@@ -423,4 +447,12 @@
       </collision>
     </link>
+    <joint name="right_hand_j15" type="revolute">
+      <axis xyz="0 1 0" />
+      <limit effort="100" velocity="${1600*M_PI/180}" lower="${-34.21*M_PI/180}" upper="${34.213*M_PI/180}" />
+      <origin xyz="0 0 -0.025" rpy="0 0 0" />
+      <parent link="pinky2"/>
+      <child link="pinky_end"/>
+    </joint>
+    <link name="pinky_end"/>
 </macro>
   <macro name="m3_r_hand" params="side parent reflect *origin">

Commit message: Added new m3openni tracker (was not working after update)+ added new kinect files for automatic calibration

File: meka_description/urdf/H2R4_r_hand_defs.urdf.xacro (robot description, xacro)
@@ -240,5 +240,5 @@
       <axis xyz="0 1 0" />
       <limit effort="100" velocity="${1600*M_PI/180}" lower="${-34.21*M_PI/180}" upper="${34.213*M_PI/180}" />
-      <origin xyz="0 0 -0.025" rpy="0 0 0" />
+      <origin xyz="0 0.008 -0.025" rpy="0 0 0" />
       <parent link="index2"/>
       <child link="index_end"/>
@@ -345,5 +345,5 @@
       <axis xyz="0 1 0" />
       <limit effort="100" velocity="${1600*M_PI/180}" lower="${-34.21*M_PI/180}" upper="${34.213*M_PI/180}" />
-      <origin xyz="0 0 -0.025" rpy="0 0 0" />
+      <origin xyz="0 0.008 -0.025" rpy="0 0 0" />
       <parent link="ring2"/>
       <child link="ring_end"/>
@@ -450,5 +450,5 @@
       <axis xyz="0 1 0" />
       <limit effort="100" velocity="${1600*M_PI/180}" lower="${-34.21*M_PI/180}" upper="${34.213*M_PI/180}" />
-      <origin xyz="0 0 -0.025" rpy="0 0 0" />
+      <origin xyz="0 0.008 -0.025" rpy="0 0 0" />
       <parent link="pinky2"/>
       <child link="pinky_end"/>
