Commit message: Added T0 in the robot description (rm from additional static transforms)

File: meka_description/urdf/Z1R2B_defs.urdf.xacro (robot description, xacro)
@@ -66,4 +66,10 @@
 	<child link="upper" />
     </joint>
+    <joint name="origin_joint" type="fixed">
+	<origin xyz="0 0 0.2337" rpy="0 0 0" />
+	<parent link="upper" />
+	<child link="T0" />
+    </joint>
+    <link name="T0"/>
   </macro>
 </robot>
