Commit message: fix j0 direction on urdf

File: meka_description/urdf/A2R4_l_arm_defs.urdf.xacro (robot description, xacro)
@@ -29,5 +29,5 @@
     <!-- Shoulder pan -->
     <joint name="left_arm_j0" type="revolute">
-      <axis xyz="0 1 0" />
+      <axis xyz="0 -1 0" />
       <insert_block name="origin" /> <!-- transform from parent link to this joint frame -->
       <parent link="${parent}"/>

Commit message: fixed lj4 joints limits

File: meka_description/urdf/A2R4_l_arm_defs.urdf.xacro (robot description, xacro)
@@ -160,5 +160,5 @@
     <joint name="left_arm_j4" type="revolute">
 	    <axis xyz="0 0 -1" />
-      <limit effort="4" velocity="${150*M_PI/180}" lower="${-19.7*M_PI/180}" upper="${199.7*M_PI/180}" />
+      <limit effort="4" velocity="${150*M_PI/180}" lower="${-190.7*M_PI/180}" upper="${19.7*M_PI/180}" />
       <origin xyz="0 0 -0.27747" rpy="0 0 0" />
       <parent link="elbowclevis_LEFT"/>
@@ -228,5 +228,5 @@
       <parent link="w_differential_LEFT"/>
       <child link="handmount_LEFT"/>
-      <dynamics damping="1.0"/>
+      <dynamics damping="0.1"/>
     </joint>
     <link name="handmount_LEFT">

Commit message: fix velocity limit on left arm

File: meka_description/urdf/A2R4_l_arm_defs.urdf.xacro (robot description, xacro)
@@ -60,5 +60,5 @@
     <joint name="left_arm_j1" type="revolute">
       <axis xyz="-1 0 0"/>
-     <limit effort="40" velocity="${30*M_PI/180}" lower="${-24*M_PI/180}" upper="${150*M_PI/180}" />
+     <limit effort="40" velocity="${30*M_PI/180}" lower="${24*M_PI/180}" upper="${-150*M_PI/180}" />
       <origin xyz="0 0 0" rpy="0 0 0" />
       <parent link="shoulderupper_LEFT"/>

Commit message: fixed joint limits on left j1

File: meka_description/urdf/A2R4_l_arm_defs.urdf.xacro (robot description, xacro)
@@ -60,5 +60,5 @@
     <joint name="left_arm_j1" type="revolute">
       <axis xyz="-1 0 0"/>
-     <limit effort="40" velocity="${30*M_PI/180}" lower="${24*M_PI/180}" upper="${-150*M_PI/180}" />
+     <limit effort="40" velocity="${30*M_PI/180}" upper="${24*M_PI/180}" lower="${-150*M_PI/180}" />
       <origin xyz="0 0 0" rpy="0 0 0" />
       <parent link="shoulderupper_LEFT"/>

Commit message: Uses mimic option to have the right number of joints (usefull for ros_control)

File: meka_description/urdf/A2R4_l_arm_defs.urdf.xacro (robot description, xacro)
@@ -1,3 +1,3 @@
-<?xml version="1.0"?>
+<?xml version="1.0" encoding="ISO-8859-1"?>
 <robot xmlns:sensor="http://playerstage.sourceforge.net/gazebo/xmlschema/#sensor"
        xmlns:controller="http://playerstage.sourceforge.net/gazebo/xmlschema/#controller"
@@ -5,4 +5,5 @@
   <property name="M_PI" value="3.1415926535897931" />
   <property name="VELOCITY_LIMIT_SCALE" value="0.6" />
+<property name="COLLISION_MESH_SCALE" value="1.0 1.0 1.0"/>
   <property name="shoulder_lift_length" value="0.10" />
   <property name="shoulder_lift_radius" value="0.12" />
@@ -54,5 +55,5 @@
 	      <origin xyz="0 0 0" rpy="${M_PI} 0.0 0.0 " />
 	      <geometry name="r_shoulder_collision_geom">
-		      <mesh filename="package://${MESH_COLL}/A2R3/A2R3_RT1_shoulderRoll.stl" />
+		      <mesh filename="package://${MESH_COLL}/A2R3/A2R3_RT1_shoulderRoll.stl"  />
 	      </geometry>
       </collision>
@@ -117,5 +118,5 @@
 	      <origin xyz="0 0 0" rpy="0.0 0.0 0.0 " />
 	      <geometry name="bicep_LEFT_geom_collision">
-		      <mesh filename="package://${MESH_COLL}/A2R3/A2R3_LT3_bicep.stl" />
+		      <mesh filename="package://${MESH_COLL}/A2R3/A2R3_LT3_bicep.stl" scale="${COLLISION_MESH_SCALE}"/>
 	      </geometry>
       </collision>
@@ -153,5 +154,5 @@
 	      <origin xyz="0 0 0" rpy="0.0 0.0 ${M_PI}" />
 	      <geometry name="elbowclevis_LEFT_collision">
-		      <mesh filename="package://${MESH_COLL}/A2R3/A2R3_RT4_elbow.stl" />
+		      <mesh filename="package://${MESH_COLL}/A2R3/A2R3_RT4_elbow.stl" scale="${COLLISION_MESH_SCALE}"/>
 	      </geometry>
       </collision>
@@ -183,5 +184,5 @@
 	      <origin xyz="0 0 0" rpy="0.0 0.0 0.0 " />
 	      <geometry name="wrist_LEFT_collision">
-		      <mesh filename="package://${MESH_COLL}/A2R3/A2R3_T5_forearmRoll.stl" />
+		      <mesh filename="package://${MESH_COLL}/A2R3/A2R3_T5_forearmRoll.stl" scale="${COLLISION_MESH_SCALE}"/>
 	      </geometry>
       </collision>
@@ -247,5 +248,5 @@
 	      <origin xyz="0 0 0" rpy="0.0 0.0 0.0 " />
 	      <geometry name="handmount_LEFT_collision">
-		      <mesh filename="package://${MESH_COLL}/A2R3/A2R3_T7_wristYaw.stl" />
+		      <mesh filename="package://${MESH_COLL}/A2R3/A2R3_T7_wristYaw.stl" scale="${COLLISION_MESH_SCALE}"/>
 	      </geometry>
       </collision>

File: meka_description/urdf/A2R4_r_arm_defs.urdf.xacro (robot description, xacro)
@@ -1,7 +1,8 @@
-<?xml version="1.0"?>
+<?xml version="1.0" encoding="ISO-8859-1"?>
 <robot xmlns:sensor="http://playerstage.sourceforge.net/gazebo/xmlschema/#sensor"
        xmlns:controller="http://playerstage.sourceforge.net/gazebo/xmlschema/#controller"
        xmlns:interface="http://playerstage.sourceforge.net/gazebo/xmlschema/#interface">
   <property name="M_PI" value="3.1415926535897931" />
+ <property name="COLLISION_MESH_SCALE" value="1.0 1.0 1.0"/>
   <macro name="m3_r_shoulder" params="side parent reflect *origin">
     <!-- Shoulder pan -->
@@ -101,5 +102,5 @@
 	      <origin xyz="0 0 0" rpy="0.0 0.0 0.0 " />
 	      <geometry name="bicep_RIGHT_geom_collision">
-		      <mesh filename="package://${MESH_COLL}/A2R3/A2R3_RT3_bicep.stl" />
+		      <mesh filename="package://${MESH_COLL}/A2R3/A2R3_RT3_bicep.stl" scale="${COLLISION_MESH_SCALE}"/>
 	      </geometry>
       </collision>
@@ -137,5 +138,5 @@
 	      <origin xyz="0 0 0" rpy="0.0 0.0 0.0 " />
 	      <geometry name="elbowclevis_RIGHT_collision">
-		      <mesh filename="package://${MESH_COLL}/A2R3/A2R3_RT4_elbow.stl" />
+		      <mesh filename="package://${MESH_COLL}/A2R3/A2R3_RT4_elbow.stl" scale="${COLLISION_MESH_SCALE}"/>
 	      </geometry>
       </collision>
@@ -170,5 +171,5 @@
 	      <origin xyz="0 0 0" rpy="0.0 0.0 0.0 " />
 	      <geometry name="wrist_RIGHT_collision">
-		      <mesh filename="package://${MESH_COLL}/A2R3/A2R3_T5_forearmRoll.stl" />
+		      <mesh filename="package://${MESH_COLL}/A2R3/A2R3_T5_forearmRoll.stl" scale="${COLLISION_MESH_SCALE}"/>
 	      </geometry>
       </collision>
@@ -234,5 +235,5 @@
 	      <origin xyz="0 0 0" rpy="0.0 0.0 0.0 " />
 	      <geometry name="handmount_RIGHT_collision">
-		      <mesh filename="package://${MESH_COLL}/A2R3/A2R3_T7_wristYaw.stl" />
+		      <mesh filename="package://${MESH_COLL}/A2R3/A2R3_T7_wristYaw.stl" scale="${COLLISION_MESH_SCALE}"/>
 	      </geometry>
       </collision>

File: meka_description/urdf/ENS_head_defs.urdf.xacro (robot description, xacro)
@@ -4,4 +4,5 @@
        xmlns:interface="http://playerstage.sourceforge.net/gazebo/xmlschema/#interface">
   <property name="M_PI" value="3.1415926535897931" />
+ <property name="EYE_LIDS_OFFSET" value="0.785" />
   <macro name="m3_neck" params="side parent reflect *origin">
     <joint name="head_j0" type="revolute">
@@ -199,8 +200,17 @@
       </collision>
     </link>
+<link name="eye_center" />
+<!--                               Eye Lids                        /-->
+<joint name="head_j7" type="revolute">
+      <axis xyz="0 1 0" />
+      <limit effort="100" velocity="${1600*M_PI/180}" lower="${35.0*M_PI/180}" upper="${78.0*M_PI/180}" />
+      <parent link="eye_tilt"/>
+      <child link="eye_center"/>
+</joint>
     <joint name="head_j7_rt_eyelid_top" type="revolute">
+<mimic joint="head_j7" multiplier="1.0" offset="-${0*M_PI/180}"/>
 	    <axis xyz="0 -1 0" />
-      <limit effort="100" velocity="${1600*M_PI/180}" lower="${2.0*M_PI/180}" upper="${68.0*M_PI/180}" />
-      <origin xyz="0 0.0 0" rpy="0 0.785 0" />
+      <limit effort="100" velocity="${1600*M_PI/180}" lower="${2.0*M_PI/180}" upper="${78.0*M_PI/180}" />
+      <origin xyz="0 0.0 0" rpy="0 ${78*M_PI/180} 0" />
       <parent link="right_eye"/>
       <child link="rt_eyelid_top"/>
@@ -222,7 +232,8 @@
     </link>
     <joint name="head_j7_rt_eyelid_bottom" type="revolute">
+	<mimic joint="head_j7" multiplier="1.0" offset="-${0*M_PI/180}"/>
 	    <axis xyz="0 1 0" />
-       <limit effort="100" velocity="${1600*M_PI/180}" lower="${2.0*M_PI/180}" upper="${68.0*M_PI/180}" />
-      <origin xyz="0 0.0 0" rpy="0 -0.785 0" />
+       <limit effort="100" velocity="${1600*M_PI/180}" lower="${2.0*M_PI/180}" upper="${78.0*M_PI/180}" />
+      <origin xyz="0 0.0 0" rpy="0 -${78*M_PI/180} 0" />
       <parent link="right_eye"/>
       <child link="rt_eyelid_bottom"/>
@@ -244,7 +255,8 @@
     </link>
     <joint name="head_j7_lt_eyelid_top" type="revolute">
+<mimic joint="head_j7" multiplier="1.0" offset="-${0*M_PI/180}"/>
 	    <axis xyz="0 -1 0" />
-       <limit effort="100" velocity="${1600*M_PI/180}" lower="${2.0*M_PI/180}" upper="${68.0*M_PI/180}" />
-      <origin xyz="0 0.0 0" rpy="0 0.785 0" />
+       <limit effort="100" velocity="${1600*M_PI/180}" lower="${2.0*M_PI/180}" upper="${78.0*M_PI/180}" />
+      <origin xyz="0 0.0 0" rpy="0 ${78*M_PI/180} 0" />
       <parent link="left_eye"/>
       <child link="lt_eyelid_top"/>
@@ -266,7 +278,8 @@
     </link>
     <joint name="head_j7_lt_eyelid_bottom" type="revolute">
+<mimic joint="head_j7" multiplier="1.0" offset="-${0*M_PI/180}"/>
 	    <axis xyz="0 1 0" />
-       <limit effort="100" velocity="${1600*M_PI/180}" lower="${2.0*M_PI/180}" upper="${68.0*M_PI/180}" />
-      <origin xyz="0 0.0 0" rpy="0 -0.785 0" />
+       <limit effort="100" velocity="${1600*M_PI/180}" lower="${2.0*M_PI/180}" upper="${78.0*M_PI/180}" />
+      <origin xyz="0 0.0 0" rpy="0 -${78*M_PI/180} 0" />
       <parent link="left_eye"/>
       <child link="lt_eyelid_bottom"/>

File: meka_description/urdf/H2R4_l_hand_defs.urdf.xacro (robot description, xacro)
@@ -3,6 +3,9 @@
        xmlns:controller="http://playerstage.sourceforge.net/gazebo/xmlschema/#controller"
        xmlns:interface="http://playerstage.sourceforge.net/gazebo/xmlschema/#interface">
-  <property name="M_PI" value="3.1415926535897931" />
-  <macro name="m3_l_palm" params="side parent reflect *origin">
+  	<property name="M_PI" value="3.1415926535897931" />
+	<property name="ndof_finger" value="3" />
+	<property name="flex_factor" value="0.3" />
+	<property name="COLLISION_MESH_SCALE" value="1.0 1.0 1.0"/>
+<macro name="m3_l_palm" params="side parent reflect *origin">
   <joint name="palm_joint_left" type="fixed">
     <origin xyz="0 0 -0.04414" rpy="0 0 0" />
@@ -31,5 +34,5 @@
 	      <origin xyz="0 0 0" rpy="0.0 0.0 0.0 " />
 	      <geometry name="palm_collision_left">
-		      <mesh filename="package://${MESH_COLL}/H2R3/H2R3_LT8_palm_left.stl" />
+		      <mesh filename="package://${MESH_COLL}/H2R3/H2R3_LT8_palm_left.stl" scale="${COLLISION_MESH_SCALE}"/>
 	      </geometry>
       </collision>
@@ -37,6 +40,6 @@
 <!-- Start Thumb -->
     <joint name="left_hand_j0" type="revolute">
-      <axis xyz="0 0 1" />
-      <origin xyz="-0.02 -0.028 -0.03" rpy="0 0 0" />
+      <axis xyz="0 0 -1" />
+      <origin xyz="-0.02 -0.028 -0.03" rpy="0 0 ${M_PI/2.0}" />
       <parent link="palm_left"/>
       <child link="thumb0_left"/>
@@ -64,5 +67,5 @@
 	      <origin xyz="0 0 0" rpy="0.0 0.0 0.0 " />
 	      <geometry name="thumb0_collision_left">
-		      <mesh filename="package://${MESH_COLL}/H2R3/H2R3_RJ0_thumb_abductlink.stl" />
+		      <mesh filename="package://${MESH_COLL}/H2R3/H2R3_RJ0_thumb_abductlink.stl" scale="${COLLISION_MESH_SCALE}"/>
 	      </geometry>
       </collision>
@@ -96,9 +99,10 @@
 	      <origin xyz="0 0 0" rpy="0.0 0.0 0.0 " />
 	      <geometry name="thumb1_collision_left">
-		      <mesh filename="package://${MESH_COLL}/H2R3/H2R3_thumb_knuckle1.stl" />
-	      </geometry>
-      </collision>
-    </link>
-    <joint name="left_hand_j2" type="revolute">
+		      <mesh filename="package://${MESH_COLL}/H2R3/H2R3_thumb_knuckle1.stl" scale="${COLLISION_MESH_SCALE}"/>
+	      </geometry>
+      </collision>
+    </link>
+    <joint name="left_hand_j1a" type="revolute">
+<mimic joint="left_hand_j1" multiplier="${flex_factor}"/>
       <axis xyz="0 -1 0" />
       <origin xyz="-0.044 0 0" rpy="0 0 0" />
@@ -128,9 +132,10 @@
 	      <origin xyz="0 0 0" rpy="0.0 0.0 0.0 " />
 	      <geometry name="thumb_knuckle2_collision_left">
-		      <mesh filename="package://${MESH_COLL}/H2R3/H2R3_thumb_knuckle2.stl" />
-	      </geometry>
-      </collision>
-    </link>
-    <joint name="left_hand_j3" type="revolute">
+		      <mesh filename="package://${MESH_COLL}/H2R3/H2R3_thumb_knuckle2.stl" scale="${COLLISION_MESH_SCALE}"/>
+	      </geometry>
+      </collision>
+    </link>
+    <joint name="left_hand_j1b" type="revolute">
+<mimic joint="left_hand_j1" multiplier="${flex_factor}"/>
       <axis xyz="0 -1 0" />
       <origin xyz="-0.035 0 0" rpy="0 0 0" />
@@ -141,7 +146,7 @@
     <link name="thumb_end_left"/>
 <!-- Start Index Finger -->
-    <joint name="left_hand_j4" type="revolute">
-      <axis xyz="0 1 0" />
-      <origin xyz="0 0.028 -0.101" rpy="0 0 0" />
+    <joint name="left_hand_j2" type="revolute">
+      <axis xyz="0 1 0" />
+      <origin xyz="0 -0.028 -0.101" rpy="0 0 0" />
       <parent link="palm_left" />
       <child link="index0_left"/>
@@ -169,9 +174,10 @@
 	      <origin xyz="0 0 0" rpy="0.0 0.0 0.0 " />
 	      <geometry name="index0_collision_left">
-		      <mesh filename="package://${MESH_COLL}/H2R3/H2R3_finger_knuckle1.stl" />
-	      </geometry>
-      </collision>
-    </link>
-    <joint name="left_hand_j5" type="revolute">
+		      <mesh filename="package://${MESH_COLL}/H2R3/H2R3_finger_knuckle1.stl" scale="${COLLISION_MESH_SCALE}"/>
+	      </geometry>
+      </collision>
+    </link>
+    <joint name="left_hand_j2a" type="revolute">
+<mimic joint="left_hand_j2" multiplier="${flex_factor}"/>
       <axis xyz="0 1 0" />
       <limit effort="100" velocity="${1600*M_PI/180}" lower="${-34.99*M_PI/180}" upper="${34.99*M_PI/180}" />
@@ -201,9 +207,10 @@
 	      <origin xyz="0 0 0" rpy="0.0 0.0 0.0 " />
 	      <geometry name="index1_collision_left">
-		      <mesh filename="package://${MESH_COLL}/H2R3/H2R3_finger_knuckle2.stl" />
-	      </geometry>
-      </collision>
-    </link>
-    <joint name="left_hand_j6" type="revolute">
+		      <mesh filename="package://${MESH_COLL}/H2R3/H2R3_finger_knuckle2.stl" scale="${COLLISION_MESH_SCALE}"/>
+	      </geometry>
+      </collision>
+    </link>
+    <joint name="left_hand_j2b" type="revolute">
+<mimic joint="left_hand_j2" multiplier="${flex_factor}"/>
       <axis xyz="0 1 0" />
       <limit effort="100" velocity="${1600*M_PI/180}" lower="${-34.21*M_PI/180}" upper="${34.213*M_PI/180}" />
@@ -233,9 +240,10 @@
 	      <origin xyz="0 0 0" rpy="0.0 0.0 0.0 " />
 	      <geometry name="index2_collision_left">
-		      <mesh filename="package://${MESH_COLL}/H2R3/H2R3_finger_knuckle3.stl" />
-	      </geometry>
-      </collision>
-    </link>
-    <joint name="left_hand_j7" type="revolute">
+		      <mesh filename="package://${MESH_COLL}/H2R3/H2R3_finger_knuckle3.stl" scale="${COLLISION_MESH_SCALE}"/>
+	      </geometry>
+      </collision>
+    </link>
+    <joint name="left_hand_j2c" type="revolute">
+<mimic joint="left_hand_j2" multiplier="${flex_factor}"/>
       <axis xyz="0 1 0" />
       <limit effort="100" velocity="${1600*M_PI/180}" lower="${-34.21*M_PI/180}" upper="${34.213*M_PI/180}" />
@@ -246,5 +254,5 @@
     <link name="index_end_left"/>
 <!-- Start Ring Finger -->
-    <joint name="left_hand_j8" type="revolute">
+    <joint name="left_hand_j3" type="revolute">
       <axis xyz="0 1 0" />
       <origin xyz="0 0 -0.101" rpy="0 0 0" />
@@ -274,9 +282,10 @@
 	      <origin xyz="0 0 0" rpy="0.0 0.0 0.0 " />
 	      <geometry name="ring0_collision_left">
-		      <mesh filename="package://${MESH_COLL}/H2R3/H2R3_finger_knuckle1.stl" />
-	      </geometry>
-      </collision>
-    </link>
-    <joint name="left_hand_j9" type="revolute">
+		      <mesh filename="package://${MESH_COLL}/H2R3/H2R3_finger_knuckle1.stl" scale="${COLLISION_MESH_SCALE}"/>
+	      </geometry>
+      </collision>
+    </link>
+    <joint name="left_hand_j3a" type="revolute">
+<mimic joint="left_hand_j3" multiplier="${flex_factor}"/>
       <axis xyz="0 1 0" />
       <limit effort="100" velocity="${1600*M_PI/180}" lower="${-34.99*M_PI/180}" upper="${34.99*M_PI/180}" />
@@ -306,9 +315,10 @@
 	      <origin xyz="0 0 0" rpy="0.0 0.0 0.0 " />
 	      <geometry name="ring1_collision_left">
-		      <mesh filename="package://${MESH_COLL}/H2R3/H2R3_finger_knuckle2.stl" />
-	      </geometry>
-      </collision>
-    </link>
-    <joint name="left_hand_j10" type="revolute">
+		      <mesh filename="package://${MESH_COLL}/H2R3/H2R3_finger_knuckle2.stl" scale="${COLLISION_MESH_SCALE}"/>
+	      </geometry>
+      </collision>
+    </link>
+    <joint name="left_hand_j3b" type="revolute">
+<mimic joint="left_hand_j3" multiplier="${flex_factor}"/>
       <axis xyz="0 1 0" />
       <limit effort="100" velocity="${1600*M_PI/180}" lower="${-34.21*M_PI/180}" upper="${34.213*M_PI/180}" />
@@ -338,9 +348,10 @@
 	      <origin xyz="0 0 0" rpy="0.0 0.0 0.0 " />
 	      <geometry name="ring2_collision_left">
-		      <mesh filename="package://${MESH_COLL}/H2R3/H2R3_finger_knuckle3.stl" />
-	      </geometry>
-      </collision>
-    </link>
-    <joint name="left_hand_j11" type="revolute">
+		      <mesh filename="package://${MESH_COLL}/H2R3/H2R3_finger_knuckle3.stl" scale="${COLLISION_MESH_SCALE}"/>
+	      </geometry>
+      </collision>
+    </link>
+    <joint name="left_hand_j3c" type="revolute">
+<mimic joint="left_hand_j3" multiplier="${flex_factor}"/>
       <axis xyz="0 1 0" />
       <limit effort="100" velocity="${1600*M_PI/180}" lower="${-34.21*M_PI/180}" upper="${34.213*M_PI/180}" />
@@ -351,7 +362,7 @@
     <link name="ring_end_left"/>
 <!-- Start Pinky Finger -->
-    <joint name="left_hand_j12" type="revolute">
-      <axis xyz="0 1 0" />
-      <origin xyz="0 -0.028 -0.101" rpy="0 0 0" />
+    <joint name="left_hand_j4" type="revolute">
+      <axis xyz="0 1 0" />
+      <origin xyz="0 0.028 -0.101" rpy="0 0 0" />
       <parent link="palm_left" />
       <child link="pinky0_left"/>
@@ -379,9 +390,10 @@
 	      <origin xyz="0 0 0" rpy="0.0 0.0 0.0 " />
 	      <geometry name="pinky0_collision_left">
-		      <mesh filename="package://${MESH_COLL}/H2R3/H2R3_finger_knuckle1.stl" />
-	      </geometry>
-      </collision>
-    </link>
-    <joint name="left_hand_j13" type="revolute">
+		      <mesh filename="package://${MESH_COLL}/H2R3/H2R3_finger_knuckle1.stl" scale="${COLLISION_MESH_SCALE}"/>
+	      </geometry>
+      </collision>
+    </link>
+    <joint name="left_hand_j4a" type="revolute">
+<mimic joint="left_hand_j4" multiplier="${flex_factor}"/>
       <axis xyz="0 1 0" />
       <limit effort="100" velocity="${1600*M_PI/180}" lower="${-34.99*M_PI/180}" upper="${34.99*M_PI/180}" />
@@ -411,9 +423,10 @@
 	      <origin xyz="0 0 0" rpy="0.0 0.0 0.0 " />
 	      <geometry name="pinky1_collision_left">
-		      <mesh filename="package://${MESH_COLL}/H2R3/H2R3_finger_knuckle2.stl" />
-	      </geometry>
-      </collision>
-    </link>
-    <joint name="left_hand_j14" type="revolute">
+		      <mesh filename="package://${MESH_COLL}/H2R3/H2R3_finger_knuckle2.stl" scale="${COLLISION_MESH_SCALE}"/>
+	      </geometry>
+      </collision>
+    </link>
+    <joint name="left_hand_j4b" type="revolute">
+<mimic joint="left_hand_j4" multiplier="${flex_factor}"/>
       <axis xyz="0 1 0" />
       <limit effort="100" velocity="${1600*M_PI/180}" lower="${-34.21*M_PI/180}" upper="${34.213*M_PI/180}" />
@@ -443,9 +456,10 @@
 	      <origin xyz="0 0 0" rpy="0.0 0.0 0.0 " />
 	      <geometry name="pinky2_collision_left">
-		      <mesh filename="package://${MESH_COLL}/H2R3/H2R3_finger_knuckle3.stl" />
-	      </geometry>
-      </collision>
-    </link>
-    <joint name="left_hand_j15" type="revolute">
+		      <mesh filename="package://${MESH_COLL}/H2R3/H2R3_finger_knuckle3.stl" scale="${COLLISION_MESH_SCALE}"/>
+	      </geometry>
+      </collision>
+    </link>
+    <joint name="left_hand_j4c" type="revolute">
+<mimic joint="left_hand_j4" multiplier="${flex_factor}"/>
       <axis xyz="0 1 0" />
       <limit effort="100" velocity="${1600*M_PI/180}" lower="${-34.21*M_PI/180}" upper="${34.213*M_PI/180}" />
