Commit message: Uses mimic option to have the right number of joints (usefull for ros_control)

File: meka_description/urdf/H2R4_r_hand_defs.urdf.xacro (robot description, xacro)
@@ -3,5 +3,8 @@
        xmlns:controller="http://playerstage.sourceforge.net/gazebo/xmlschema/#controller"
        xmlns:interface="http://playerstage.sourceforge.net/gazebo/xmlschema/#interface">
-  <property name="M_PI" value="3.1415926535897931" />
+<property name="M_PI" value="3.1415926535897931" />
+<property name="ndof_finger" value="3" />
+<property name="flex_factor" value="0.5" />
+<property name="COLLISION_MESH_SCALE" value="1.0 1.0 1.0"/>
   <macro name="m3_r_palm" params="side parent reflect *origin">
   <joint name="palm_joint_right" type="fixed">
@@ -31,5 +34,5 @@
 	      <origin xyz="0 0 0" rpy="0.0 0.0 0.0 " />
 	      <geometry name="palm_collision_right">
-		      <mesh filename="package://${MESH_COLL}/H2R3/H2R3_RT8_palm_right.stl" />
+		      <mesh filename="package://${MESH_COLL}/H2R3/H2R3_RT8_palm_right.stl" scale="${COLLISION_MESH_SCALE}"/>
 	      </geometry>
       </collision>
@@ -37,9 +40,9 @@
 <!-- Start Thumb -->
     <joint name="right_hand_j0" type="revolute">
-      <axis xyz="0 0 -1" />
-      <origin xyz="-0.02 0.028 -0.03" rpy="0 0 0" />
+      <axis xyz="0 0 1" />
+      <origin xyz="-0.02 0.028 -0.03" rpy="0 0 -${M_PI/2.0}" />
       <parent link="palm_right"/>
       <child link="thumb0_right"/>
-      <limit effort="100" velocity="${20.0*M_PI/180}" lower="${-40*M_PI/180}" upper="${15*M_PI/180}" />
+      <limit effort="100" velocity="${20.0*M_PI/180}" lower="${0*M_PI/180}" upper="${130*M_PI/180}" />
     </joint>
     <link name="thumb0_right">
@@ -64,5 +67,5 @@
 	      <origin xyz="0 0 0" rpy="0.0 0.0 0.0 " />
 	      <geometry name="thumb0_collision_right">
-		      <mesh filename="package://${MESH_COLL}/H2R3/H2R3_RJ0_thumb_abductlink.stl" />
+		      <mesh filename="package://${MESH_COLL}/H2R3/H2R3_RJ0_thumb_abductlink.stl" scale="${COLLISION_MESH_SCALE}"/>
 	      </geometry>
       </collision>
@@ -70,5 +73,5 @@
     <joint name="right_hand_j1" type="revolute">
       <axis xyz="0 -1 0"/>
-     <limit effort="100" velocity="${75*M_PI/180}" lower="${-80.919*M_PI/180}" upper="${80.91*M_PI/180}" />
+     <limit effort="100" velocity="${75*M_PI/180}" lower="${0*M_PI/180}" upper="${189*M_PI/180}" />
       <origin xyz="-0.018 0 0" rpy="0 0 0" />
       <parent link="thumb0_right"/>
@@ -96,9 +99,10 @@
 	      <origin xyz="0 0 0" rpy="0.0 0.0 0.0 " />
 	      <geometry name="thumb1_collision_right">
-		      <mesh filename="package://${MESH_COLL}/H2R3/H2R3_thumb_knuckle1.stl" />
-	      </geometry>
-      </collision>
-    </link>
-    <joint name="right_hand_j2" type="revolute">
+		      <mesh filename="package://${MESH_COLL}/H2R3/H2R3_thumb_knuckle1.stl" scale="${COLLISION_MESH_SCALE}"/>
+	      </geometry>
+      </collision>
+    </link>
+    <joint name="right_hand_j1a" type="revolute">
+	<mimic joint="right_hand_j1" multiplier="${flex_factor}"/>
       <axis xyz="0 -1 0" />
       <origin xyz="-0.044 0 0" rpy="0 0 0" />
@@ -128,9 +132,10 @@
 	      <origin xyz="0 0 0" rpy="0.0 0.0 0.0 " />
 	      <geometry name="thumb_knuckle2_collision_right">
-		      <mesh filename="package://${MESH_COLL}/H2R3/H2R3_thumb_knuckle2.stl" />
-	      </geometry>
-      </collision>
-    </link>
-    <joint name="right_hand_j3" type="revolute">
+		      <mesh filename="package://${MESH_COLL}/H2R3/H2R3_thumb_knuckle2.stl" scale="${COLLISION_MESH_SCALE}"/>
+	      </geometry>
+      </collision>
+    </link>
+    <joint name="right_hand_j1b" type="revolute">
+<mimic joint="right_hand_j1" multiplier="${flex_factor}"/>
       <axis xyz="0 -1 0" />
       <origin xyz="-0.035 0 0" rpy="0 0 0" />
@@ -141,10 +146,10 @@
     <link name="thumb_end_right"/>
 <!-- Start Index Finger -->
-    <joint name="right_hand_j4" type="revolute">
+    <joint name="right_hand_j2" type="revolute">
       <axis xyz="0 1 0" />
       <origin xyz="0 0.028 -0.101" rpy="0 0 0" />
       <parent link="palm_right" />
       <child link="index0_right"/>
-	<limit effort="100" velocity="${50*M_PI/180}" lower="${-7.072*M_PI/180}" upper="${37.072*M_PI/180}" />
+	<limit effort="100" velocity="${50*M_PI/180}" lower="${0*M_PI/180}" upper="${276*M_PI/180}" />
     </joint>
     <link name="index0_right">
@@ -169,9 +174,10 @@
 	      <origin xyz="0 0 0" rpy="0.0 0.0 0.0 " />
 	      <geometry name="index0_collision_right">
-		      <mesh filename="package://${MESH_COLL}/H2R3/H2R3_finger_knuckle1.stl" />
-	      </geometry>
-      </collision>
-    </link>
-    <joint name="right_hand_j5" type="revolute">
+		      <mesh filename="package://${MESH_COLL}/H2R3/H2R3_finger_knuckle1.stl" scale="${COLLISION_MESH_SCALE}"/>
+	      </geometry>
+      </collision>
+    </link>
+    <joint name="right_hand_j2a" type="revolute">
+<mimic joint="right_hand_j2" multiplier="${flex_factor}"/>
       <axis xyz="0 1 0" />
       <limit effort="100" velocity="${1600*M_PI/180}" lower="${-34.99*M_PI/180}" upper="${34.99*M_PI/180}" />
@@ -201,9 +207,10 @@
 	      <origin xyz="0 0 0" rpy="0.0 0.0 0.0 " />
 	      <geometry name="index1_collision_right">
-		      <mesh filename="package://${MESH_COLL}/H2R3/H2R3_finger_knuckle2.stl" />
-	      </geometry>
-      </collision>
-    </link>
-    <joint name="right_hand_j6" type="revolute">
+		      <mesh filename="package://${MESH_COLL}/H2R3/H2R3_finger_knuckle2.stl" scale="${COLLISION_MESH_SCALE}"/>
+	      </geometry>
+      </collision>
+    </link>
+    <joint name="right_hand_j2b" type="revolute">
+<mimic joint="right_hand_j2" multiplier="${flex_factor}"/>
       <axis xyz="0 1 0" />
       <limit effort="100" velocity="${1600*M_PI/180}" lower="${-34.21*M_PI/180}" upper="${34.213*M_PI/180}" />
@@ -233,9 +240,10 @@
 	      <origin xyz="0 0 0" rpy="0.0 0.0 0.0 " />
 	      <geometry name="index2_collision_right">
-		      <mesh filename="package://${MESH_COLL}/H2R3/H2R3_finger_knuckle3.stl" />
-	      </geometry>
-      </collision>
-    </link>
-    <joint name="right_hand_j7" type="revolute">
+		      <mesh filename="package://${MESH_COLL}/H2R3/H2R3_finger_knuckle3.stl" scale="${COLLISION_MESH_SCALE}"/>
+	      </geometry>
+      </collision>
+    </link>
+    <joint name="right_hand_j2c" type="revolute">
+<mimic joint="right_hand_j2" multiplier="${flex_factor}"/>
       <axis xyz="0 1 0" />
       <limit effort="100" velocity="${1600*M_PI/180}" lower="${-34.21*M_PI/180}" upper="${34.213*M_PI/180}" />
@@ -246,5 +254,5 @@
     <link name="index_end_right"/>
 <!-- Start Ring Finger -->
-    <joint name="right_hand_j8" type="revolute">
+    <joint name="right_hand_j3" type="revolute">
       <axis xyz="0 1 0" />
       <origin xyz="0 0 -0.101" rpy="0 0 0" />
@@ -274,9 +282,10 @@
 	      <origin xyz="0 0 0" rpy="0.0 0.0 0.0 " />
 	      <geometry name="ring0_collision_right">
-		      <mesh filename="package://${MESH_COLL}/H2R3/H2R3_finger_knuckle1.stl" />
-	      </geometry>
-      </collision>
-    </link>
-    <joint name="right_hand_j9" type="revolute">
+		      <mesh filename="package://${MESH_COLL}/H2R3/H2R3_finger_knuckle1.stl" scale="${COLLISION_MESH_SCALE}"/>
+	      </geometry>
+      </collision>
+    </link>
+    <joint name="right_hand_j3a" type="revolute">
+<mimic joint="right_hand_j3" multiplier="${flex_factor}"/>
       <axis xyz="0 1 0" />
       <limit effort="100" velocity="${1600*M_PI/180}" lower="${-34.99*M_PI/180}" upper="${34.99*M_PI/180}" />
@@ -306,9 +315,10 @@
 	      <origin xyz="0 0 0" rpy="0.0 0.0 0.0 " />
 	      <geometry name="ring1_collision_right">
-		      <mesh filename="package://${MESH_COLL}/H2R3/H2R3_finger_knuckle2.stl" />
-	      </geometry>
-      </collision>
-    </link>
-    <joint name="right_hand_j10" type="revolute">
+		      <mesh filename="package://${MESH_COLL}/H2R3/H2R3_finger_knuckle2.stl" scale="${COLLISION_MESH_SCALE}"/>
+	      </geometry>
+      </collision>
+    </link>
+    <joint name="right_hand_j3b" type="revolute">
+<mimic joint="right_hand_j3" multiplier="${flex_factor}"/>
       <axis xyz="0 1 0" />
       <limit effort="100" velocity="${1600*M_PI/180}" lower="${-34.21*M_PI/180}" upper="${34.213*M_PI/180}" />
@@ -338,9 +348,10 @@
 	      <origin xyz="0 0 0" rpy="0.0 0.0 0.0 " />
 	      <geometry name="ring2_collision_right">
-		      <mesh filename="package://${MESH_COLL}/H2R3/H2R3_finger_knuckle3.stl" />
-	      </geometry>
-      </collision>
-    </link>
-    <joint name="right_hand_j11" type="revolute">
+		      <mesh filename="package://${MESH_COLL}/H2R3/H2R3_finger_knuckle3.stl" scale="${COLLISION_MESH_SCALE}"/>
+	      </geometry>
+      </collision>
+    </link>
+    <joint name="right_hand_j3c" type="revolute">
+<mimic joint="right_hand_j3" multiplier="${flex_factor}"/>
       <axis xyz="0 1 0" />
       <limit effort="100" velocity="${1600*M_PI/180}" lower="${-34.21*M_PI/180}" upper="${34.213*M_PI/180}" />
@@ -351,5 +362,5 @@
     <link name="ring_end_right"/>
 <!-- Start Pinky Finger -->
-    <joint name="right_hand_j12" type="revolute">
+    <joint name="right_hand_j4" type="revolute">
       <axis xyz="0 1 0" />
       <origin xyz="0 -0.028 -0.101" rpy="0 0 0" />
@@ -379,9 +390,10 @@
 	      <origin xyz="0 0 0" rpy="0.0 0.0 0.0 " />
 	      <geometry name="pinky0_collision_right">
-		      <mesh filename="package://${MESH_COLL}/H2R3/H2R3_finger_knuckle1.stl" />
-	      </geometry>
-      </collision>
-    </link>
-    <joint name="right_hand_j13" type="revolute">
+		      <mesh filename="package://${MESH_COLL}/H2R3/H2R3_finger_knuckle1.stl" scale="${COLLISION_MESH_SCALE}"/>
+	      </geometry>
+      </collision>
+    </link>
+    <joint name="right_hand_j4a" type="revolute">
+<mimic joint="right_hand_j4" multiplier="${flex_factor}"/>
       <axis xyz="0 1 0" />
       <limit effort="100" velocity="${1600*M_PI/180}" lower="${-34.99*M_PI/180}" upper="${34.99*M_PI/180}" />
@@ -411,9 +423,10 @@
 	      <origin xyz="0 0 0" rpy="0.0 0.0 0.0 " />
 	      <geometry name="pinky1_collision_right">
-		      <mesh filename="package://${MESH_COLL}/H2R3/H2R3_finger_knuckle2.stl" />
-	      </geometry>
-      </collision>
-    </link>
-    <joint name="right_hand_j14" type="revolute">
+		      <mesh filename="package://${MESH_COLL}/H2R3/H2R3_finger_knuckle2.stl" scale="${COLLISION_MESH_SCALE}"/>
+	      </geometry>
+      </collision>
+    </link>
+    <joint name="right_hand_j4b" type="revolute">
+<mimic joint="right_hand_j4" multiplier="${flex_factor}"/>
       <axis xyz="0 1 0" />
       <limit effort="100" velocity="${1600*M_PI/180}" lower="${-34.21*M_PI/180}" upper="${34.213*M_PI/180}" />
@@ -443,9 +456,10 @@
 	      <origin xyz="0 0 0" rpy="0.0 0.0 0.0 " />
 	      <geometry name="pinky2_collision_right">
-		      <mesh filename="package://${MESH_COLL}/H2R3/H2R3_finger_knuckle3.stl" />
-	      </geometry>
-      </collision>
-    </link>
-    <joint name="right_hand_j15" type="revolute">
+		      <mesh filename="package://${MESH_COLL}/H2R3/H2R3_finger_knuckle3.stl" scale="${COLLISION_MESH_SCALE}"/>
+	      </geometry>
+      </collision>
+    </link>
+    <joint name="right_hand_j4c" type="revolute">
+<mimic joint="right_hand_j4" multiplier="${flex_factor}"/>
       <axis xyz="0 1 0" />
       <limit effort="100" velocity="${1600*M_PI/180}" lower="${-34.21*M_PI/180}" upper="${34.213*M_PI/180}" />

File: meka_description/urdf/S2R1B_head_defs.urdf.xacro (robot description, xacro)
@@ -200,5 +200,13 @@
       </collision>
     </link>
+<joint name="head_j7" type="revolute">
+      <axis xyz="0 1 0" />
+      <limit effort="100" velocity="${1600*M_PI/180}" lower="${2.0*M_PI/180}" upper="${68.0*M_PI/180}" />
+      <origin xyz="0 0.008 -0.025" rpy="0 0 0" />
+      <parent link="right_eye"/>
+      <child link="rt_eyelid_top"/>
+</joint>
     <joint name="head_j7_rt_eyelid_top" type="revolute">
+<mimic joint="head_j7" multiplier="1.0" offset="-${35*M_PI/180}"/>
 	    <axis xyz="0 -1 0" />
       <limit effort="100" velocity="${1600*M_PI/180}" lower="${2.0*M_PI/180}" upper="${68.0*M_PI/180}" />
@@ -223,4 +231,5 @@
     </link>
     <joint name="head_j7_rt_eyelid_bottom" type="revolute">
+	<mimic joint="head_j7" multiplier="1.0" offset="-${35*M_PI/180}"/>
 	    <axis xyz="0 1 0" />
        <limit effort="100" velocity="${1600*M_PI/180}" lower="${2.0*M_PI/180}" upper="${68.0*M_PI/180}" />
@@ -245,4 +254,5 @@
     </link>
     <joint name="head_j7_lt_eyelid_top" type="revolute">
+<mimic joint="head_j7" multiplier="1.0" offset="-${35*M_PI/180}"/>
 	    <axis xyz="0 -1 0" />
        <limit effort="100" velocity="${1600*M_PI/180}" lower="${2.0*M_PI/180}" upper="${68.0*M_PI/180}" />
@@ -267,4 +277,5 @@
     </link>
     <joint name="head_j7_lt_eyelid_bottom" type="revolute">
+<mimic joint="head_j7" multiplier="1.0" offset="-${35*M_PI/180}"/>
 	    <axis xyz="0 1 0" />
        <limit effort="100" velocity="${1600*M_PI/180}" lower="${2.0*M_PI/180}" upper="${68.0*M_PI/180}" />
@@ -288,4 +299,5 @@
       </collision>
     </link>
+ <!-- Ears
      <joint name="head_j8" type="revolute">
 	    <axis xyz="0 0 1" />
@@ -376,4 +388,5 @@
       </collision>
     </link>
+/-->
 </macro>
   <macro name="m3_head" params="side parent reflect *origin">
