Commit message: Updated URDFs to work with groovy

File: meka_description/robots/ens.urdf.xacro (robot description, xacro)
@@ -17,8 +17,10 @@
 <!-- Meka Arm -->
   <include filename="$(find meka_description)/urdf/A2R4_r_arm_defs.urdf.xacro" />
+  <include filename="$(find meka_description)/urdf/A2R4_l_arm_defs.urdf.xacro" />
   <!-- Meka Hand -->
   <include filename="$(find meka_description)/urdf/H2R4_r_hand_defs.urdf.xacro" />
+  <include filename="$(find meka_description)/urdf/H2R4_l_hand_defs.urdf.xacro" />
 <!-- Meka Head -->
-  <include filename="$(find meka_description)/urdf/S2R1B_head_defs.urdf.xacro" />
+  <include filename="$(find meka_description)/urdf/ENS_head_defs.urdf.xacro" />
   <!-- john added transmissions -->
   <include filename="$(find meka_description)/transmissions/A2R4_r_arm_defs.transmission.xacro" />
@@ -41,4 +43,7 @@
     <origin xyz="0.0 0.0 0.0" rpy="0 0 0" />
   </m3_r_hand>
+  <!--<m3_l_hand side="l" reflect="1" parent="handmount_LEFT">
+    <origin xyz="0.0 0.0 0.0" rpy="0 0 0" />
+  </m3_l_hand>-->
   <m3_head side="r" reflect="1" parent="upper">
     <origin xyz="0.0 0.0 0.31155" rpy="0 0 0" />
@@ -47,7 +52,10 @@
     <origin xyz="0.0 -0.18465 0.2337" rpy="0 0 0" />
   </m3_r_arm>
+ <!--<m3_l_arm side="l" reflect="1" parent="upper">
+    <origin xyz="0.0 0.18465 0.2337" rpy="0 0 0" />
+  </m3_l_arm>-->
   <link name="world" />
   <link name="base_link" />
-<!-- Solid Base -->
+  <!-- Solid Base -->
   <joint name="base_joint" type="fixed">
 	  <origin xyz="0 0 1" rpy="0 0 0" />
@@ -63,5 +71,5 @@
   <!-- Solid Base -->
   <joint name="chest_joint" type="fixed">
-	  <origin xyz="0 0 0.0" rpy="0 0 0" />
+	  <origin xyz="0 0 -0.03" rpy="0 0 0" />
     <parent link="zlift_link" />
     <child link="upper" />
@@ -77,11 +85,12 @@
 		  <origin xyz="0 0 0" rpy="0 0 0" />
 		  <geometry name="upper_geom">
-			  <mesh filename="package://${MESH}/T2R3/T2R3_TJ3_chest_waist_neck.dae" />
+			  <mesh filename="package://${MESH}/A2R3/A2R3_T4_Chest_Neck.dae" />
 		  </geometry>
+		  <material name="Blue" />
 	  </visual>
 	  <collision>
 		  <origin xyz="0 0 0" rpy="0.0 0.0 0.0 " />
 		  <geometry name="upper_collision_geom">
-			  <mesh filename="package://${MESH_COLL}/T2R3/T2R3_TJ3_chest_waist_neck.stl" />
+			  <mesh filename="package://${MESH_COLL}/A2R3/A2R3_T4_Chest_Neck.stl" />
 		  </geometry>
 	  </collision>

File: meka_description/robots/gai.urdf.xacro (robot description, xacro)
@@ -6,31 +6,25 @@
        name="meka" >
  <property name="M_PI" value="3.1415926535897931" />
- <property name="R_ARM" value="ma16" />
- <property name="R_HAND" value="mh12" />
- <property name="L_ARM" value="ma17" />
- <property name="L_HAND" value="mh13" />
- <property name="TORSO" value="mt5" />
-  <property name="HEAD" value="ms2" />
  <property name="MESH" value="meka_description/meshes/mid_res" />
  <property name="MESH_COLL" value="meka_description/meshes/low_res" />
 <!-- generic simulator_gazebo plugins for starting mechanism control, ros time, ros battery -->
   <include filename="$(find meka_description)/gazebo/gazebo.urdf.xacro" />
-  <include filename="$(find meka_description)/transmissions/uta.transmission.xacro" />
+  <!--<include filename="$(find meka_description)/transmissions/uta.transmission.xacro" />-->
 <!-- Meka Base -->
-  <include filename="$(find meka_description)/urdf/B1R2_defs.urdf.xacro" />
+  <include filename="$(find meka_description)/urdf/B1R2B_defs.urdf.xacro" />
 <!-- Meka Zlift -->
-  <include filename="$(find meka_description)/urdf/Z1R2_defs.urdf.xacro" />
+  <include filename="$(find meka_description)/urdf/Z1R2B_defs.urdf.xacro" />
 <!-- Meka Arm -->
-  <include filename="$(find meka_description)/urdf/A2R3_r_arm_defs.urdf.xacro" />
-  <include filename="$(find meka_description)/urdf/A2R3_l_arm_defs.urdf.xacro" />
+  <include filename="$(find meka_description)/urdf/A2R4_r_arm_defs.urdf.xacro" />
+  <include filename="$(find meka_description)/urdf/A2R4_l_arm_defs.urdf.xacro" />
   <!-- Meka Hand -->
-  <include filename="$(find meka_description)/urdf/H2R2_r_hand_defs.urdf.xacro" />
-  <include filename="$(find meka_description)/urdf/H2R2_l_hand_defs.urdf.xacro" />
+  <include filename="$(find meka_description)/urdf/H2R4_r_hand_defs.urdf.xacro" />
+ <!--<include filename="$(find meka_description)/urdf/H2R4_l_hand_defs.urdf.xacro" />-->
 <!-- Meka Head -->
-  <include filename="$(find meka_description)/urdf/S2R1_head_defs.urdf.xacro" />
+<!--<include filename="$(find meka_description)/urdf/SIMC_head_defs.urdf.xacro" />-->
   <!-- john added transmissions -->
-  <include filename="$(find meka_description)/transmissions/A2R3_r_arm_defs.transmission.xacro" />
-  <include filename="$(find meka_description)/transmissions/H2R2_r_hand_defs.transmission.xacro" />
-  <include filename="$(find meka_description)/transmissions/S2R1_head_defs.transmission.xacro" />
+  <include filename="$(find meka_description)/transmissions/A2R4_r_arm_defs.transmission.xacro" />
+  <!--<include filename="$(find meka_description)/transmissions/H2R2_r_hand_defs.transmission.xacro" />-->
+  <!--<include filename="$(find meka_description)/transmissions/S2R1_head_defs.transmission.xacro" />-->
    <property name="M_PI" value="3.1415926535897931" />
   <material name="GreyA"> <!-- darkest -->
@@ -49,16 +43,19 @@
     <origin xyz="0.0 0.0 0.0" rpy="0 0 0" />
   </m3_r_hand>
+  <!--<m3_l_hand side="l" reflect="1" parent="handmount_LEFT">
+    <origin xyz="0.0 0.0 0.0" rpy="0 0 0" />
+  </m3_l_hand>-->
   <m3_head side="r" reflect="1" parent="upper">
     <origin xyz="0.0 0.0 0.31155" rpy="0 0 0" />
   </m3_head>
-  <!--<m3_l_arm side="l" reflect="1" parent="upper">
-    <origin xyz="0.0 0.18465 0.2337" rpy="0 0 0" />
-  </m3_l_arm>-->
  <m3_r_arm side="r" reflect="1" parent="upper">
     <origin xyz="0.0 -0.18465 0.2337" rpy="0 0 0" />
   </m3_r_arm>
+ <m3_l_arm side="l" reflect="1" parent="upper">
+    <origin xyz="0.0 0.18465 0.2337" rpy="0 0 0" />
+  </m3_l_arm>
   <link name="world" />
   <link name="base_link" />
-<!-- Solid Base -->
+  <!-- Solid Base -->
   <joint name="base_joint" type="fixed">
 	  <origin xyz="0 0 1" rpy="0 0 0" />
@@ -74,5 +71,5 @@
   <!-- Solid Base -->
   <joint name="chest_joint" type="fixed">
-	  <origin xyz="0 0 0.0" rpy="0 0 0" />
+	  <origin xyz="0 0 -0.03" rpy="0 0 0" />
     <parent link="zlift_link" />
     <child link="upper" />
@@ -88,11 +85,12 @@
 		  <origin xyz="0 0 0" rpy="0 0 0" />
 		  <geometry name="upper_geom">
-			  <mesh filename="package://${MESH}/T2R3/T2R3_TJ3_chest_waist_neck.dae" />
+			  <mesh filename="package://${MESH}/A2R3/A2R3_T4_Chest_Neck.dae" />
 		  </geometry>
+		  <material name="Blue" />
 	  </visual>
 	  <collision>
 		  <origin xyz="0 0 0" rpy="0.0 0.0 0.0 " />
 		  <geometry name="upper_collision_geom">
-			  <mesh filename="package://${MESH_COLL}/T2R3/T2R3_TJ3_chest_waist_neck.stl" />
+			  <mesh filename="package://${MESH_COLL}/A2R3/A2R3_T4_Chest_Neck.stl" />
 		  </geometry>
 	  </collision>

File: meka_description/robots/m1.urdf.xacro (robot description, xacro)
@@ -71,5 +71,5 @@
   <!-- Solid Base -->
   <joint name="chest_joint" type="fixed">
-	  <origin xyz="0 0 0.0" rpy="0 0 0" />
+	  <origin xyz="0 0 -0.03" rpy="0 0 0" />
     <parent link="zlift_link" />
     <child link="upper" />
@@ -85,6 +85,7 @@
 		  <origin xyz="0 0 0" rpy="0 0 0" />
 		  <geometry name="upper_geom">
-			  <mesh filename="package://${MESH}/T2R3/T2R3_TJ3_chest_waist_neck.dae" />
+			  <mesh filename="package://${MESH}/A2R3/A2R3_T4_Chest_Neck.dae" />
 		  </geometry>
+		  <material name="Blue" />
 	  </visual>
 	  <collision>

File: meka_description/robots/simc.urdf.xacro (robot description, xacro)
@@ -6,31 +6,25 @@
        name="meka" >
  <property name="M_PI" value="3.1415926535897931" />
- <property name="R_ARM" value="ma16" />
- <property name="R_HAND" value="mh12" />
- <property name="L_ARM" value="ma17" />
- <property name="L_HAND" value="mh13" />
- <property name="TORSO" value="mt5" />
-  <property name="HEAD" value="ms2" />
  <property name="MESH" value="meka_description/meshes/mid_res" />
  <property name="MESH_COLL" value="meka_description/meshes/low_res" />
 <!-- generic simulator_gazebo plugins for starting mechanism control, ros time, ros battery -->
   <include filename="$(find meka_description)/gazebo/gazebo.urdf.xacro" />
-  <include filename="$(find meka_description)/transmissions/uta.transmission.xacro" />
+  <!--<include filename="$(find meka_description)/transmissions/uta.transmission.xacro" />-->
 <!-- Meka Base -->
-  <include filename="$(find meka_description)/urdf/B1R2_defs.urdf.xacro" />
+  <include filename="$(find meka_description)/urdf/B1R2B_defs.urdf.xacro" />
 <!-- Meka Zlift -->
-  <include filename="$(find meka_description)/urdf/Z1R2_defs.urdf.xacro" />
+  <include filename="$(find meka_description)/urdf/Z1R2B_defs.urdf.xacro" />
 <!-- Meka Arm -->
-  <include filename="$(find meka_description)/urdf/A2R3_r_arm_defs.urdf.xacro" />
-  <include filename="$(find meka_description)/urdf/A2R3_l_arm_defs.urdf.xacro" />
+  <include filename="$(find meka_description)/urdf/A2R4_r_arm_defs.urdf.xacro" />
+  <include filename="$(find meka_description)/urdf/A2R4_l_arm_defs.urdf.xacro" />
   <!-- Meka Hand -->
-  <include filename="$(find meka_description)/urdf/H2R2_r_hand_defs.urdf.xacro" />
-  <include filename="$(find meka_description)/urdf/H2R2_l_hand_defs.urdf.xacro" />
+  <include filename="$(find meka_description)/urdf/H2R4_r_hand_defs.urdf.xacro" />
+  <include filename="$(find meka_description)/urdf/H2R4_l_hand_defs.urdf.xacro" />
 <!-- Meka Head -->
-  <include filename="$(find meka_description)/urdf/S2R1_head_defs.urdf.xacro" />
+  <include filename="$(find meka_description)/urdf/SIMC_head_defs.urdf.xacro" />
   <!-- john added transmissions -->
-  <include filename="$(find meka_description)/transmissions/A2R3_r_arm_defs.transmission.xacro" />
-  <include filename="$(find meka_description)/transmissions/H2R2_r_hand_defs.transmission.xacro" />
-  <include filename="$(find meka_description)/transmissions/S2R1_head_defs.transmission.xacro" />
+  <include filename="$(find meka_description)/transmissions/A2R4_r_arm_defs.transmission.xacro" />
+  <!--<include filename="$(find meka_description)/transmissions/H2R2_r_hand_defs.transmission.xacro" />-->
+  <!--<include filename="$(find meka_description)/transmissions/S2R1_head_defs.transmission.xacro" />-->
    <property name="M_PI" value="3.1415926535897931" />
   <material name="GreyA"> <!-- darkest -->
@@ -49,16 +43,19 @@
     <origin xyz="0.0 0.0 0.0" rpy="0 0 0" />
   </m3_r_hand>
+  <m3_l_hand side="l" reflect="1" parent="handmount_LEFT">
+    <origin xyz="0.0 0.0 0.0" rpy="0 0 0" />
+  </m3_l_hand>
   <m3_head side="r" reflect="1" parent="upper">
     <origin xyz="0.0 0.0 0.31155" rpy="0 0 0" />
   </m3_head>
-  <!--<m3_l_arm side="l" reflect="1" parent="upper">
-    <origin xyz="0.0 0.18465 0.2337" rpy="0 0 0" />
-  </m3_l_arm>-->
  <m3_r_arm side="r" reflect="1" parent="upper">
     <origin xyz="0.0 -0.18465 0.2337" rpy="0 0 0" />
   </m3_r_arm>
+ <m3_l_arm side="l" reflect="1" parent="upper">
+    <origin xyz="0.0 0.18465 0.2337" rpy="0 0 0" />
+  </m3_l_arm>
   <link name="world" />
   <link name="base_link" />
-<!-- Solid Base -->
+  <!-- Solid Base -->
   <joint name="base_joint" type="fixed">
 	  <origin xyz="0 0 1" rpy="0 0 0" />
@@ -74,5 +71,5 @@
   <!-- Solid Base -->
   <joint name="chest_joint" type="fixed">
-	  <origin xyz="0 0 0.0" rpy="0 0 0" />
+	  <origin xyz="0 0 -0.03" rpy="0 0 0" />
     <parent link="zlift_link" />
     <child link="upper" />
@@ -88,11 +85,12 @@
 		  <origin xyz="0 0 0" rpy="0 0 0" />
 		  <geometry name="upper_geom">
-			  <mesh filename="package://${MESH}/T2R3/T2R3_TJ3_chest_waist_neck.dae" />
+			  <mesh filename="package://${MESH}/A2R3/A2R3_T4_Chest_Neck.dae" />
 		  </geometry>
+		  <material name="Blue" />
 	  </visual>
 	  <collision>
 		  <origin xyz="0 0 0" rpy="0.0 0.0 0.0 " />
 		  <geometry name="upper_collision_geom">
-			  <mesh filename="package://${MESH_COLL}/T2R3/T2R3_TJ3_chest_waist_neck.stl" />
+			  <mesh filename="package://${MESH_COLL}/A2R3/A2R3_T4_Chest_Neck.stl" />
 		  </geometry>
 	  </collision>

File: meka_description/urdf/A2R4_l_arm_defs.urdf.xacro (robot description, xacro)
@@ -33,6 +33,5 @@
       <parent link="${parent}"/>
       <child link="shoulderupper_LEFT"/>
-      <limit lower="${reflect*M_PI/4-1.5}"  upper="${reflect*M_PI/4+1.5}"
-             effort="30" velocity="${VELOCITY_LIMIT_SCALE*3.48}" />
+      <limit effort="40" velocity="${30.0*M_PI/180}" lower="${-80*M_PI/180}" upper="${200*M_PI/180}" />
       <dynamics damping="10.0" />
       <safety_controller k_position="100" k_velocity="10"
@@ -67,6 +66,5 @@
       <axis xyz="-1 0 0"/>
       <!-- Limits updated from Function's CAD values as of 2009_02_24 (link_data.xls) -->
-      <limit lower="-0.5236" upper="1.3963"
-             effort="30" velocity="${VELOCITY_LIMIT_SCALE*3.47}" />
+      <limit effort="40" velocity="${30*M_PI/180}" upper="${24*M_PI/180}"  lower="${-150*M_PI/180}" />
       <safety_controller k_position="100" k_velocity="10"
                          soft_lower_limit="${-0.5236+0.17}" soft_upper_limit="${1.3963-0.05}" />
@@ -104,5 +102,5 @@
       <parent link="shoulderpitch_LEFT" />
       <child link="bicep_LEFT"/>
-      <limit lower="${reflect*1.55-2.35}" upper="${reflect*1.55+2.35}" effort="30" velocity="${VELOCITY_LIMIT_SCALE*5.45}" />
+     <limit effort="20" velocity="${50*M_PI/180}" lower="${-85*M_PI/180}" upper="${85*M_PI/180}" />
       <safety_controller k_position="100" k_velocity="2" soft_lower_limit="${reflect*1.55-2.35+0.15}" soft_upper_limit="${reflect*1.55+2.35-0.15}" />
       <dynamics damping="0.1" />
@@ -139,6 +137,5 @@
       <parent link="${parent}"/>
       <child link="elbowclevis_LEFT"/>
-	<limit lower="${reflect*M_PI/4-1.5}"  upper="${reflect*M_PI/4+1.5}"
-             effort="30" velocity="${VELOCITY_LIMIT_SCALE*3.48}" />
+	<limit effort="20" velocity="${50*M_PI/180}" lower="${-0.278978*M_PI/180}" upper="${132.8175*M_PI/180}" />
     </joint>
     <link name="elbowclevis_LEFT">
@@ -156,7 +153,7 @@
       <visual>
 	      <material name="GreyA" />
-	      <origin xyz="0 0 0" rpy="0 0 0 " />
+	      <origin xyz="0 0 0" rpy="0 0 3.14 " />
 	      <geometry name="elbowclevis_LEFT_geom">
-		      <mesh filename="package://${MESH}/A2R3/A2R3_LT4_elbow.dae" />
+		      <mesh filename="package://${MESH}/A2R3/A2R3_RT4_elbow.dae" />
 	      </geometry>
       </visual>
@@ -171,5 +168,5 @@
     <joint name="left_arm_j4" type="revolute">
 	    <axis xyz="0 0 -1" />
-      <limit lower="-2.3" upper="0.1" effort="30" velocity="${VELOCITY_LIMIT_SCALE*5.5}" />
+     <limit effort="4" velocity="${150*M_PI/180}" lower="${-190.7*M_PI/180}" upper="${19.7*M_PI/180}" />
       <safety_controller k_position="100" k_velocity="3" soft_lower_limit="${-2.3+0.25}" soft_upper_limit="${0.1-0.1}" />
       <dynamics damping="1.0" />
@@ -208,6 +205,5 @@
       <parent link="${parent}"/>
       <child link="w_differential_LEFT"/>
-	<limit lower="${reflect*M_PI/4-1.5}"  upper="${reflect*M_PI/4+1.5}"
-             effort="30" velocity="${VELOCITY_LIMIT_SCALE*3.48}" />
+	<limit effort="8" velocity="${40*M_PI/180}" lower="${-58.83*M_PI/180}" upper="${58.83*M_PI/180}" />
     </joint>
     <link name="w_differential_LEFT">
@@ -236,5 +232,5 @@
     <joint name="left_arm_j6" type="revolute">
 	    <axis xyz="-1 0 0" />
-      <limit lower="-0.1" upper="2.2" effort="200" velocity="${VELOCITY_LIMIT_SCALE*5.13}" />
+      <limit effort="8" velocity="${40*M_PI/180}" lower="${-60*M_PI/180}" upper="${60*M_PI/180}" />
       <safety_controller k_position="20" k_velocity="4" soft_lower_limit="${-0.1+0.2}" soft_upper_limit="${2.2-0.2}" />
       <dynamics damping="0.1" />
