Commit message: Updated URDFs to work with groovy

File: meka_description/urdf/S2R1B_head_defs.urdf.xacro (robot description, xacro)
@@ -10,5 +10,5 @@
       <parent link="${parent}"/>
       <child link="neck_tilt"/>
-      <limit effort="100" velocity="${20.0*M_PI/180}" lower="${-40*M_PI/180}" upper="${15*M_PI/180}" />
+      <limit effort="100" velocity="${20.0*M_PI/180}" lower="${-18.0*M_PI/180}" upper="${1.0*M_PI/180}" />
     </joint>
     <link name="neck_tilt">
@@ -39,5 +39,5 @@
     <joint name="head_j1" type="revolute">
       <axis xyz="0 0 1"/>
-     <limit effort="100" velocity="${75*M_PI/180}" lower="${-80.919*M_PI/180}" upper="${80.91*M_PI/180}" />
+     <limit effort="100" velocity="${75*M_PI/180}" lower="${-56.0*M_PI/180}" upper="${56.0*M_PI/180}" />
       <origin xyz="0 0 0.13849" rpy="0 0 0" />
       <parent link="neck_tilt"/>
@@ -74,5 +74,5 @@
       <parent link="neck_roll" />
       <child link="neck_yaw"/>
-      <limit effort="100" velocity="${50*M_PI/180}" lower="${-14.94*M_PI/180}" upper="${14.94*M_PI/180}" />
+      <limit effort="100" velocity="${50*M_PI/180}" lower="${-15.87*M_PI/180}" upper="${15.87*M_PI/180}" />
     </joint>
     <link name="neck_yaw">
@@ -101,10 +101,10 @@
       </collision>
     </link>
-      <joint name="head_j3" type="revolute">
+    <joint name="head_j3" type="revolute">
 		  <axis xyz="0 -1 0" />
       <origin xyz="0 0 0" rpy="0 0 0" />
       <parent link="neck_yaw" />
       <child link="head_shell"/>
-	<limit effort="100" velocity="${50*M_PI/180}" lower="${-7.072*M_PI/180}" upper="${37.072*M_PI/180}" />
+	<limit effort="100" velocity="${50*M_PI/180}" lower="${-8.0*M_PI/180}" upper="${-2.0*M_PI/180}" />
     </joint>
     <link name="head_shell">
@@ -123,5 +123,6 @@
 	      <origin xyz="0 0 0" rpy="0 0 0 " />
 	      <geometry name="head_shell_geom">
-		      <mesh filename="package://${MESH}/S2R1/S2R1_H4_UTA_head.dae" />
+		<mesh filename="package://${MESH}/S2R1/S2R1_H4_SIMC_head.dae" />
+		<!--<mesh filename="package://${MESH}/S2R1/S2R1_H4_UTA_head.dae" />-->
 	      </geometry>
       </visual>
@@ -129,5 +130,5 @@
 	      <origin xyz="0 0 0" rpy="0.0 0.0 0.0 " />
 	      <geometry name="head_shell_collision">
-		      <mesh filename="package://${MESH_COLL}/S2R1/S2R1_H4_UTA_head.stl" />
+		      <mesh filename="package://${MESH_COLL}/S2R1/S2R1_H4_SIMC_head.stl" />
 	      </geometry>
       </collision>
@@ -135,5 +136,5 @@
     <joint name="head_j4" type="revolute">
 	    <axis xyz="0 -1 0" />
-      <limit effort="100" velocity="${1600*M_PI/180}" lower="${-34.99*M_PI/180}" upper="${34.99*M_PI/180}" />
+      <limit effort="100" velocity="${1600*M_PI/180}" lower="${-70.1*M_PI/180}" upper="${70.1*M_PI/180}" />
       <origin xyz="0.12508 0 0" rpy="0 0 0" />
       <parent link="head_shell"/>
@@ -157,5 +158,5 @@
     <joint name="head_j5" type="revolute">
 	    <axis xyz="0 0 1" />
-      <limit effort="100" velocity="${1600*M_PI/180}" lower="${-34.21*M_PI/180}" upper="${34.213*M_PI/180}" />
+      <limit effort="100" velocity="${1600*M_PI/180}" lower="${-37.49*M_PI/180}" upper="${37.4*M_PI/180}" />
       <origin xyz="0 -0.053 0" rpy="0 0 0" />
       <parent link="eye_tilt"/>
@@ -179,5 +180,5 @@
     <joint name="head_j6" type="revolute">
 	    <axis xyz="0 0 1" />
-      <limit effort="100" velocity="${1600*M_PI/180}" lower="${-35.12*M_PI/180}" upper="${35.125*M_PI/180}" />
+      <limit effort="100" velocity="${1600*M_PI/180}" lower="${-37.9*M_PI/180}" upper="${37.99*M_PI/180}" />
       <origin xyz="0 0.053 0" rpy="0 0 0" />
       <parent link="eye_tilt"/>
@@ -196,4 +197,180 @@
 	      <geometry name="left_eye_collision">
 		      <mesh filename="package://${MESH_COLL}/S2R1/S2R1_eye.stl" />
+	      </geometry>
+      </collision>
+    </link>
+    <joint name="head_j7_rt_eyelid_top" type="revolute">
+	    <axis xyz="0 -1 0" />
+      <limit effort="100" velocity="${1600*M_PI/180}" lower="${2.0*M_PI/180}" upper="${68.0*M_PI/180}" />
+      <origin xyz="0 0.0 0" rpy="0 0.785 0" />
+      <parent link="right_eye"/>
+      <child link="rt_eyelid_top"/>
+    </joint>
+    <link name="rt_eyelid_top">
+      <visual>
+	      <material name="GreyC" />
+	      <origin xyz="0 0 0" rpy="0 0 0 " />
+	      <geometry name="rt_eyelid_top_geom">
+		      <mesh filename="package://${MESH}/S2R1/eyelid_top.dae" />
+	      </geometry>
+      </visual>
+      <collision>
+	      <origin xyz="0 0 0" rpy="0.0 0.0 0.0 " />
+	      <geometry name="rt_eyelid_top_collision">
+		      <box size="0.01 0.01 0.01" />
+	      </geometry>
+      </collision>
+    </link>
+    <joint name="head_j7_rt_eyelid_bottom" type="revolute">
+	    <axis xyz="0 1 0" />
+       <limit effort="100" velocity="${1600*M_PI/180}" lower="${2.0*M_PI/180}" upper="${68.0*M_PI/180}" />
+      <origin xyz="0 0.0 0" rpy="0 -0.785 0" />
+      <parent link="right_eye"/>
+      <child link="rt_eyelid_bottom"/>
+    </joint>
+    <link name="rt_eyelid_bottom">
+      <visual>
+	      <material name="GreyC" />
+	      <origin xyz="0 0 0" rpy="0 0 0 " />
+	      <geometry name="eyelid_bottom_geom">
+		      <mesh filename="package://${MESH}/S2R1/eyelid_bottom.dae" />
+	      </geometry>
+      </visual>
+      <collision>
+	      <origin xyz="0 0 0" rpy="0.0 0.0 0.0 " />
+	      <geometry name="eyelid_bottom_collision">
+		      <box size="0.01 0.01 0.01" />
+	      </geometry>
+      </collision>
+    </link>
+    <joint name="head_j7_lt_eyelid_top" type="revolute">
+	    <axis xyz="0 -1 0" />
+       <limit effort="100" velocity="${1600*M_PI/180}" lower="${2.0*M_PI/180}" upper="${68.0*M_PI/180}" />
+      <origin xyz="0 0.0 0" rpy="0 0.785 0" />
+      <parent link="left_eye"/>
+      <child link="lt_eyelid_top"/>
+    </joint>
+    <link name="lt_eyelid_top">
+      <visual>
+	      <material name="GreyC" />
+	      <origin xyz="0 0 0" rpy="0 0 0 " />
+	      <geometry name="lt_eyelid_top_geom">
+		      <mesh filename="package://${MESH}/S2R1/eyelid_top.dae" />
+	      </geometry>
+      </visual>
+      <collision>
+	      <origin xyz="0 0 0" rpy="0.0 0.0 0.0 " />
+	      <geometry name="lt_eyelid_top_collision">
+		      <box size="0.01 0.01 0.01" />
+	      </geometry>
+      </collision>
+    </link>
+    <joint name="head_j7_lt_eyelid_bottom" type="revolute">
+	    <axis xyz="0 1 0" />
+       <limit effort="100" velocity="${1600*M_PI/180}" lower="${2.0*M_PI/180}" upper="${68.0*M_PI/180}" />
+      <origin xyz="0 0.0 0" rpy="0 -0.785 0" />
+      <parent link="left_eye"/>
+      <child link="lt_eyelid_bottom"/>
+    </joint>
+    <link name="lt_eyelid_bottom">
+      <visual>
+	      <material name="GreyC" />
+	      <origin xyz="0 0 0" rpy="0 0 0 " />
+	      <geometry name="eyelid_bottom_geom2">
+		      <mesh filename="package://${MESH}/S2R1/eyelid_bottom.dae" />
+	      </geometry>
+      </visual>
+      <collision>
+	      <origin xyz="0 0 0" rpy="0.0 0.0 0.0 " />
+	      <geometry name="eyelid_bottom_collision2">
+		      <box size="0.01 0.01 0.01" />
+	      </geometry>
+      </collision>
+    </link>
+     <joint name="head_j8" type="revolute">
+	    <axis xyz="0 0 1" />
+      <limit effort="100" velocity="${1600*M_PI/180}" lower="${-150.0*M_PI/180}" upper="${150.0*M_PI/180}" />
+      <origin xyz="0.022 0.138 0.120" rpy="-1.13 0 0" />
+      <parent link="head_shell"/>
+      <child link="ear_roll"/>
+    </joint>
+    <link name="ear_roll">
+      <visual>
+	      <material name="GreyC" />
+	      <origin xyz="0 0 0" rpy="0 0 0 " />
+	      <geometry name="ear_roll_geom">
+		      <mesh filename="package://${MESH}/S2R1/ear_mount.dae" />
+	      </geometry>
+      </visual>
+      <collision>
+	      <origin xyz="0 0 0" rpy="0.0 0.0 0.0 " />
+	      <geometry name="ear_roll_collision">
+		      <box size="0.01 0.01 0.01" />
+	      </geometry>
+      </collision>
+    </link>
+    <joint name="head_j9" type="revolute">
+	    <axis xyz="0 -1 0" />
+      <limit effort="100" velocity="${1600*M_PI/180}" lower="${0.0*M_PI/180}" upper="${123.0*M_PI/180}" />
+      <origin xyz="0.0 0.0 0.0" rpy="0 1.07 0" />
+      <parent link="ear_roll"/>
+      <child link="ear1"/>
+    </joint>
+    <link name="ear1">
+      <visual>
+	      <material name="GreyC" />
+	      <origin xyz="0 0 0" rpy="0 0 0 " />
+	      <geometry name="ear1_geom">
+		      <mesh filename="package://${MESH}/S2R1/ear.dae" />
+	      </geometry>
+      </visual>
+      <collision>
+	      <origin xyz="0 0 0" rpy="0.0 0.0 0.0 " />
+	      <geometry name="ear1_collision">
+		      <box size="0.01 0.01 0.01" />
+	      </geometry>
+      </collision>
+    </link>
+    <joint name="head_j10" type="revolute">
+	    <axis xyz="0 0 1" />
+       <limit effort="100" velocity="${1600*M_PI/180}" lower="${-150.0*M_PI/180}" upper="${150.0*M_PI/180}" />
+      <origin xyz="0.022 -0.138 0.120" rpy="1.13 0 0" />
+      <parent link="head_shell"/>
+      <child link="ear_roll2"/>
+    </joint>
+    <link name="ear_roll2">
+      <visual>
+	      <material name="GreyC" />
+	      <origin xyz="0 0 0" rpy="0 0 0 " />
+	      <geometry name="ear_roll_geom2">
+		      <mesh filename="package://${MESH}/S2R1/ear_mount.dae" />
+	      </geometry>
+      </visual>
+      <collision>
+	      <origin xyz="0 0 0" rpy="0.0 0.0 0.0 " />
+	      <geometry name="ear_roll_collision2">
+		      <box size="0.01 0.01 0.01" />
+	      </geometry>
+      </collision>
+    </link>
+    <joint name="head_j11" type="revolute">
+	    <axis xyz="0 -1 0" />
+     <limit effort="100" velocity="${1600*M_PI/180}" lower="${0.0*M_PI/180}" upper="${123.0*M_PI/180}" />
+      <origin xyz="0.0 0.0 0.0" rpy="0 1.07 0" />
+      <parent link="ear_roll2"/>
+      <child link="ear2"/>
+    </joint>
+    <link name="ear2">
+      <visual>
+	      <material name="GreyC" />
+	      <origin xyz="0 0 0" rpy="0 0 0 " />
+	      <geometry name="ear2_geom">
+		      <mesh filename="package://${MESH}/S2R1/ear.dae" />
+	      </geometry>
+      </visual>
+      <collision>
+	      <origin xyz="0 0 0" rpy="0.0 0.0 0.0 " />
+	      <geometry name="ear2_collision">
+		      <box size="0.01 0.01 0.01" />
 	      </geometry>
       </collision>

File: meka_description/urdf/Z1R2B_defs.urdf.xacro (robot description, xacro)
@@ -11,5 +11,5 @@
       <parent link="${parent}"/>
       <child link="zlift_link"/>
-      <limit lower="${reflect*M_PI/4-1.5}"  upper="${reflect*M_PI/4+1.5}"
+      <limit lower="${0.0*M_PI/180.0}"  upper="${31965.0*M_PI/180.0}"
              effort="30" velocity="${3.48}" />
       <dynamics damping="10.0" />
@@ -36,5 +36,5 @@
 	      <origin xyz="0 0 0" rpy="0.0 0.0 0.0 " />
 	      <geometry name="z_lift_geom_collision_geom">
-		      <box size="0.01 0.01 0.01" />
+		      <mesh filename="package://${MESH_COLL}/B1R1/MB1_00_011_festo-chest_mount_assy+spacer.stl" />
 	      </geometry>
       </collision>

Commit message: Added Moveit! config pkg+Updated meka urdf (eyelids)+updated joint_state_publisher

File: meka_description/robots/ens.urdf.xacro (robot description, xacro)
@@ -9,6 +9,21 @@
  <property name="MESH_COLL" value="meka_description/meshes/low_res" />
 <!-- generic simulator_gazebo plugins for starting mechanism control, ros time, ros battery -->
-  <include filename="$(find meka_description)/gazebo/gazebo.urdf.xacro" />
-  <!--<include filename="$(find meka_description)/transmissions/uta.transmission.xacro" />-->
+ <include filename="$(find meka_description)/gazebo/gazebo.urdf.xacro" />
+ <!--<include filename="$(find meka_description)/transmissions/uta.transmission.xacro" />-->
+ <link name="world" />
+ <link name="base_link" />
+ <!-- Solid Base -->
+ <joint name="base_joint" type="fixed">
+  <origin xyz="0 0 1" rpy="0 0 0" />
+  <parent link="world" />
+  <child link="base_link" />
+ </joint>
+  <xacro:meka_base  side="r" reflect="1" parent="base_link">
+    <origin xyz="0.0 0.0 0.0" rpy="0 0 0" />
+  </xacro:meka_base>
+  <xacro:meka_zlift  side="r" reflect="1" parent="dummy_3">
+    <origin xyz="0.43 0.0 0.75" rpy="0 0 0" />
+  </xacro:meka_zlift>
+  <!-- Solid Base -->
 <!-- Meka Base -->
   <include filename="$(find meka_description)/urdf/B1R2B_defs.urdf.xacro" />
@@ -38,61 +53,20 @@
   </material>
   <!-- john added transmissions -->
-  <m3_r_arm_transmission side="r" reflect="1" parent="upper"/>
-  <m3_r_hand_transmission/>
-  <m3_r_hand side="r" reflect="1" parent="handmount_RIGHT">
+  <xacro:m3_r_arm_transmission side="r" reflect="1" parent="upper"/>
+  <!--</m3_r_hand_transmission-->
+  <xacro:m3_r_hand side="r" reflect="1" parent="handmount_RIGHT">
     <origin xyz="0.0 0.0 0.0" rpy="0 0 0" />
-  </m3_r_hand>
+  </xacro:m3_r_hand>
   <!--<m3_l_hand side="l" reflect="1" parent="handmount_LEFT">
     <origin xyz="0.0 0.0 0.0" rpy="0 0 0" />
   </m3_l_hand>-->
-  <m3_head side="r" reflect="1" parent="upper">
+  <xacro:m3_head side="r" reflect="1" parent="upper">
     <origin xyz="0.0 0.0 0.31155" rpy="0 0 0" />
-  </m3_head>
- <m3_r_arm side="r" reflect="1" parent="upper">
+  </xacro:m3_head>
+ <xacro:m3_r_arm side="r" reflect="1" parent="upper">
     <origin xyz="0.0 -0.18465 0.2337" rpy="0 0 0" />
-  </m3_r_arm>
+  </xacro:m3_r_arm>
  <!--<m3_l_arm side="l" reflect="1" parent="upper">
     <origin xyz="0.0 0.18465 0.2337" rpy="0 0 0" />
   </m3_l_arm>-->
-  <link name="world" />
-  <link name="base_link" />
-  <!-- Solid Base -->
-  <joint name="base_joint" type="fixed">
-	  <origin xyz="0 0 1" rpy="0 0 0" />
-    <parent link="world" />
-    <child link="base_link" />
-  </joint>
-  <meka_base  side="r" reflect="1" parent="base_link">
-    <origin xyz="0.0 0.0 0.0" rpy="0 0 0" />
-  </meka_base>
-  <meka_zlift  side="r" reflect="1" parent="dummy_3">
-    <origin xyz="0.43 0.0 0.75" rpy="0 0 0" />
-  </meka_zlift>
-  <!-- Solid Base -->
-  <joint name="chest_joint" type="fixed">
-	  <origin xyz="0 0 -0.03" rpy="0 0 0" />
-    <parent link="zlift_link" />
-    <child link="upper" />
-  </joint>
-  <link name="upper">
-	  <inertial>
-		  <mass value="1000" />
-		  <origin xyz="0 0 0" />
-		  <inertia ixx="1000"  ixy="0"  ixz="0" iyy="1000" iyz="0" izz="1000" />
-	  </inertial>
-	  <visual>
-		  <material name="GreyC" />
-		  <origin xyz="0 0 0" rpy="0 0 0" />
-		  <geometry name="upper_geom">
-			  <mesh filename="package://${MESH}/A2R3/A2R3_T4_Chest_Neck.dae" />
-		  </geometry>
-		  <material name="Blue" />
-	  </visual>
-	  <collision>
-		  <origin xyz="0 0 0" rpy="0.0 0.0 0.0 " />
-		  <geometry name="upper_collision_geom">
-			  <mesh filename="package://${MESH_COLL}/A2R3/A2R3_T4_Chest_Neck.stl" />
-		  </geometry>
-	  </collision>
-  </link>
 </robot>

File: meka_description/urdf/ENS_head_defs.urdf.xacro (robot description, xacro)
@@ -120,5 +120,5 @@
       </inertial>
       <visual>
-	      <material name="GreyA" />
+	      <material name="GreyC" />
 	      <origin xyz="0 0 0" rpy="0 0 0 " />
 	      <geometry name="head_shell_geom">
@@ -196,4 +196,92 @@
 	      <geometry name="left_eye_collision">
 		      <mesh filename="package://${MESH_COLL}/S2R1/S2R1_eye.stl" />
+	      </geometry>
+      </collision>
+    </link>
+    <joint name="head_j7_rt_eyelid_top" type="revolute">
+	    <axis xyz="0 -1 0" />
+      <limit effort="100" velocity="${1600*M_PI/180}" lower="${2.0*M_PI/180}" upper="${68.0*M_PI/180}" />
+      <origin xyz="0 0.0 0" rpy="0 0.785 0" />
+      <parent link="right_eye"/>
+      <child link="rt_eyelid_top"/>
+    </joint>
+    <link name="rt_eyelid_top">
+      <visual>
+	      <material name="GreyC" />
+	      <origin xyz="0 0 0" rpy="0 0 0 " />
+	      <geometry name="rt_eyelid_top_geom">
+		      <mesh filename="package://${MESH}/S2R1/eyelid_top.dae" />
+	      </geometry>
+      </visual>
+      <collision>
+	      <origin xyz="0 0 0" rpy="0.0 0.0 0.0 " />
+	      <geometry name="rt_eyelid_top_collision">
+		      <box size="0.01 0.01 0.01" />
+	      </geometry>
+      </collision>
+    </link>
+    <joint name="head_j7_rt_eyelid_bottom" type="revolute">
+	    <axis xyz="0 1 0" />
+       <limit effort="100" velocity="${1600*M_PI/180}" lower="${2.0*M_PI/180}" upper="${68.0*M_PI/180}" />
+      <origin xyz="0 0.0 0" rpy="0 -0.785 0" />
+      <parent link="right_eye"/>
+      <child link="rt_eyelid_bottom"/>
+    </joint>
+    <link name="rt_eyelid_bottom">
+      <visual>
+	      <material name="GreyC" />
+	      <origin xyz="0 0 0" rpy="0 0 0 " />
+	      <geometry name="eyelid_bottom_geom">
+		      <mesh filename="package://${MESH}/S2R1/eyelid_bottom.dae" />
+	      </geometry>
+      </visual>
+      <collision>
+	      <origin xyz="0 0 0" rpy="0.0 0.0 0.0 " />
+	      <geometry name="eyelid_bottom_collision">
+		      <box size="0.01 0.01 0.01" />
+	      </geometry>
+      </collision>
+    </link>
+    <joint name="head_j7_lt_eyelid_top" type="revolute">
+	    <axis xyz="0 -1 0" />
+       <limit effort="100" velocity="${1600*M_PI/180}" lower="${2.0*M_PI/180}" upper="${68.0*M_PI/180}" />
+      <origin xyz="0 0.0 0" rpy="0 0.785 0" />
+      <parent link="left_eye"/>
+      <child link="lt_eyelid_top"/>
+    </joint>
+    <link name="lt_eyelid_top">
+      <visual>
+	      <material name="GreyC" />
+	      <origin xyz="0 0 0" rpy="0 0 0 " />
+	      <geometry name="lt_eyelid_top_geom">
+		      <mesh filename="package://${MESH}/S2R1/eyelid_top.dae" />
+	      </geometry>
+      </visual>
+      <collision>
+	      <origin xyz="0 0 0" rpy="0.0 0.0 0.0 " />
+	      <geometry name="lt_eyelid_top_collision">
+		      <box size="0.01 0.01 0.01" />
+	      </geometry>
+      </collision>
+    </link>
+    <joint name="head_j7_lt_eyelid_bottom" type="revolute">
+	    <axis xyz="0 1 0" />
+       <limit effort="100" velocity="${1600*M_PI/180}" lower="${2.0*M_PI/180}" upper="${68.0*M_PI/180}" />
+      <origin xyz="0 0.0 0" rpy="0 -0.785 0" />
+      <parent link="left_eye"/>
+      <child link="lt_eyelid_bottom"/>
+    </joint>
+    <link name="lt_eyelid_bottom">
+      <visual>
+	      <material name="GreyC" />
+	      <origin xyz="0 0 0" rpy="0 0 0 " />
+	      <geometry name="eyelid_bottom_geom2">
+		      <mesh filename="package://${MESH}/S2R1/eyelid_bottom.dae" />
+	      </geometry>
+      </visual>
+      <collision>
+	      <origin xyz="0 0 0" rpy="0.0 0.0 0.0 " />
+	      <geometry name="eyelid_bottom_collision2">
+		      <box size="0.01 0.01 0.01" />
 	      </geometry>
       </collision>

File: meka_description/urdf/Z1R2B_defs.urdf.xacro (robot description, xacro)
@@ -40,4 +40,30 @@
       </collision>
     </link>
+  <link name="upper">
+	  <inertial>
+		  <mass value="1000" />
+		  <origin xyz="0 0 0" />
+		  <inertia ixx="1000"  ixy="0"  ixz="0" iyy="1000" iyz="0" izz="1000" />
+	  </inertial>
+	  <visual>
+		  <material name="GreyC" />
+		  <origin xyz="0 0 0" rpy="0 0 0" />
+		  <geometry name="upper_geom">
+			  <mesh filename="package://${MESH}/A2R3/A2R3_T4_Chest_Neck.dae" />
+		  </geometry>
+		  <!--material name="Blue" /-->
+	  </visual>
+	  <collision>
+		  <origin xyz="0 0 0" rpy="0.0 0.0 0.0 " />
+		  <geometry name="upper_collision_geom">
+			  <mesh filename="package://${MESH_COLL}/A2R3/A2R3_T4_Chest_Neck.stl" />
+		  </geometry>
+	  </collision>
+  </link>
+    <joint name="chest_joint" type="fixed">
+	<origin xyz="0 0 -0.03" rpy="0 0 0" />
+	<parent link="zlift_link" />
+	<child link="upper" />
+    </joint>
   </macro>
 </robot>
