Commit message: Added left arm/hand URDF

File: meka_description/robots/ens.urdf.xacro (robot description, xacro)
@@ -54,11 +54,12 @@
   <!-- john added transmissions -->
   <xacro:m3_r_arm_transmission side="r" reflect="1" parent="upper"/>
+  <xacro:m3_l_arm_transmission side="r" reflect="1" parent="upper"/>
   <!--</m3_r_hand_transmission-->
   <xacro:m3_r_hand side="r" reflect="1" parent="handmount_RIGHT">
     <origin xyz="0.0 0.0 0.0" rpy="0 0 0" />
   </xacro:m3_r_hand>
-  <!--<m3_l_hand side="l" reflect="1" parent="handmount_LEFT">
+  <xacro:m3_l_hand side="l" reflect="1" parent="handmount_LEFT">
     <origin xyz="0.0 0.0 0.0" rpy="0 0 0" />
-  </m3_l_hand>-->
+  </xacro:m3_l_hand>
   <xacro:m3_head side="r" reflect="1" parent="upper">
     <origin xyz="0.0 0.0 0.31155" rpy="0 0 0" />
@@ -67,6 +68,6 @@
     <origin xyz="0.0 -0.18465 0.2337" rpy="0 0 0" />
   </xacro:m3_r_arm>
- <!--<m3_l_arm side="l" reflect="1" parent="upper">
+ <xacro:m3_l_arm side="l" reflect="1" parent="upper">
     <origin xyz="0.0 0.18465 0.2337" rpy="0 0 0" />
-  </m3_l_arm>-->
+  </xacro:m3_l_arm>
 </robot>

File: meka_description/urdf/A2R4_l_arm_defs.urdf.xacro (robot description, xacro)
@@ -29,5 +29,5 @@
     <!-- Shoulder pan -->
     <joint name="left_arm_j0" type="revolute">
-      <axis xyz="0 -1 0" />
+      <axis xyz="0 1 0" />
       <insert_block name="origin" /> <!-- transform from parent link to this joint frame -->
       <parent link="${parent}"/>

File: meka_description/urdf/H2R4_l_hand_defs.urdf.xacro (robot description, xacro)
@@ -5,10 +5,10 @@
   <property name="M_PI" value="3.1415926535897931" />
   <macro name="m3_l_palm" params="side parent reflect *origin">
-  <joint name="l_palm_joint" type="fixed">
+  <joint name="palm_joint_left" type="fixed">
     <origin xyz="0 0 -0.04414" rpy="0 0 0" />
     <parent link="${parent}"/>
-    <child link="l_palm" />
+    <child link="palm_left" />
   </joint>
-     <link name="l_palm">
+     <link name="palm_left">
       <inertial>
         <mass value="0.663" />
@@ -22,7 +22,7 @@
       </inertial>
       <visual>
-	      <material name="GreyA" />
-	      <origin xyz="0 0 0" rpy="0 0 0 " />
-	      <geometry name="l_palm_geom">
+	      <material name="GreyC" />
+	      <origin xyz="0 0 0" rpy="0 0 0 " />
+	      <geometry name="palm_geom_left">
 		      <mesh filename="package://${MESH}/H2R3/H2R3_LT8_palm_left.dae" />
 	      </geometry>
@@ -30,6 +30,6 @@
       <collision>
 	      <origin xyz="0 0 0" rpy="0.0 0.0 0.0 " />
-	      <geometry name="l_palm_collision">
-		      <mesh filename="package://${MESH_COLL}/H2R3/H2R3_RT8_palm_right.stl" />
+	      <geometry name="palm_collision_left">
+		      <mesh filename="package://${MESH_COLL}/H2R3/H2R3_LT8_palm_left.dae" />
 	      </geometry>
       </collision>
@@ -37,11 +37,11 @@
 <!-- Start Thumb -->
     <joint name="left_hand_j0" type="revolute">
-      <axis xyz="0 0 -1" />
+      <axis xyz="0 0 1" />
       <origin xyz="-0.02 -0.028 -0.03" rpy="0 0 0" />
-      <parent link="l_palm"/>
-      <child link="l_thumb0"/>
+      <parent link="palm_left"/>
+      <child link="thumb0_left"/>
       <limit effort="100" velocity="${20.0*M_PI/180}" lower="${-40*M_PI/180}" upper="${15*M_PI/180}" />
     </joint>
-    <link name="l_thumb0">
+    <link name="thumb0_left">
       <inertial>
         <mass value="0.0117" />
@@ -57,5 +57,5 @@
 	      <material name="GreyA" />
 	      <origin xyz="0 0 0" rpy="0 0 0 " />
-	      <geometry name="l_thumb0_geom">
+	      <geometry name="thumb0_geom_left">
 		      <mesh filename="package://${MESH}/H2R3/H2R3_RJ0_thumb_abductlink.dae" />
 	      </geometry>
@@ -63,5 +63,5 @@
       <collision>
 	      <origin xyz="0 0 0" rpy="0.0 0.0 0.0 " />
-	      <geometry name="l_thumb0_collision">
+	      <geometry name="thumb0_collision_left">
 		      <mesh filename="package://${MESH_COLL}/H2R3/H2R3_RJ0_thumb_abductlink.stl" />
 	      </geometry>
@@ -72,8 +72,8 @@
      <limit effort="100" velocity="${75*M_PI/180}" lower="${-80.919*M_PI/180}" upper="${80.91*M_PI/180}" />
       <origin xyz="-0.018 0 0" rpy="0 0 0" />
-      <parent link="l_thumb0"/>
-      <child link="l_thumb1"/>
-    </joint>
-    <link name="l_thumb1">
+      <parent link="thumb0_left"/>
+      <child link="thumb1_left"/>
+    </joint>
+    <link name="thumb1_left">
       <inertial>
         <mass value="0.0344" />
@@ -89,5 +89,5 @@
 	      <material name="GreyB" />
 	      <origin xyz="0 0 0" rpy="0 0 0 " />
-	      <geometry name="l_thumb1_geom">
+	      <geometry name="thumb1_geom_left">
 		      <mesh filename="package://${MESH}/H2R3/H2R3_thumb_knuckle1.dae" />
 	      </geometry>
@@ -95,5 +95,5 @@
       <collision>
 	      <origin xyz="0 0 0" rpy="0.0 0.0 0.0 " />
-	      <geometry name="l_thumb1_collision">
+	      <geometry name="thumb1_collision_left">
 		      <mesh filename="package://${MESH_COLL}/H2R3/H2R3_thumb_knuckle1.stl" />
 	      </geometry>
@@ -103,23 +103,23 @@
       <axis xyz="0 -1 0" />
       <origin xyz="-0.044 0 0" rpy="0 0 0" />
-      <parent link="l_thumb1" />
-      <child link="l_thumb2"/>
+      <parent link="thumb1_left" />
+      <child link="thumb2_left"/>
       <limit effort="100" velocity="${50*M_PI/180}" lower="${-14.94*M_PI/180}" upper="${14.94*M_PI/180}" />
     </joint>
-    <link name="l_thumb2">
-      <inertial>
-        <mass value="0.01" />
-	<origin xyz="0.0 0.0 0.0"/>
-	<inertia ixx="0.0"
-	iyy="0.0"
-	izz="0.0"
-	ixy="0.0"
-	ixz="0.0"
-	iyz="0.0" />
-      </inertial>
-      <visual>
-	      <material name="GreyC" />
-	      <origin xyz="0 0 0" rpy="0 0 0 " />
-	      <geometry name="l_thumb_knuckle2_geom">
+    <link name="thumb2_left">
+      <inertial>
+        <mass value="0.01" />
+	<origin xyz="0.0 0.0 0.0"/>
+	<inertia ixx="0.0"
+	iyy="0.0"
+	izz="0.0"
+	ixy="0.0"
+	ixz="0.0"
+	iyz="0.0" />
+      </inertial>
+      <visual>
+	      <material name="GreyC" />
+	      <origin xyz="0 0 0" rpy="0 0 0 " />
+	      <geometry name="thumb_knuckle2_geom_left">
 		      <mesh filename="package://${MESH}/H2R3/H2R3_thumb_knuckle2.dae" />
 	      </geometry>
@@ -127,18 +127,26 @@
       <collision>
 	      <origin xyz="0 0 0" rpy="0.0 0.0 0.0 " />
-	      <geometry name="l_thumb_knuckle2_collision">
+	      <geometry name="thumb_knuckle2_collision_left">
 		      <mesh filename="package://${MESH_COLL}/H2R3/H2R3_thumb_knuckle2.stl" />
 	      </geometry>
       </collision>
     </link>
+    <joint name="left_hand_j3" type="revolute">
+      <axis xyz="0 -1 0" />
+      <origin xyz="-0.035 0 0" rpy="0 0 0" />
+      <parent link="thumb2_left" />
+      <child link="thumb_end_left"/>
+      <limit effort="100" velocity="${50*M_PI/180}" lower="${-14.94*M_PI/180}" upper="${14.94*M_PI/180}" />
+    </joint>
+    <link name="thumb_end_left"/>
 <!-- Start Index Finger -->
-    <joint name="left_hand_j3" type="revolute">
+    <joint name="left_hand_j4" type="revolute">
       <axis xyz="0 1 0" />
       <origin xyz="0 0.028 -0.101" rpy="0 0 0" />
-      <parent link="l_palm" />
-      <child link="l_index0"/>
+      <parent link="palm_left" />
+      <child link="index0_left"/>
 	<limit effort="100" velocity="${50*M_PI/180}" lower="${-7.072*M_PI/180}" upper="${37.072*M_PI/180}" />
     </joint>
-    <link name="l_index0">
+    <link name="index0_left">
       <inertial>
         <mass value="0.01" />
@@ -154,5 +162,5 @@
 	      <material name="GreyA" />
 	      <origin xyz="0 0 0" rpy="0 0 0 " />
-	      <geometry name="l_index0_geom">
+	      <geometry name="index0_geom_left">
 		     <mesh filename="package://${MESH}/H2R3/H2R3_finger_knuckle1.dae" />
 	      </geometry>
@@ -160,17 +168,17 @@
       <collision>
 	      <origin xyz="0 0 0" rpy="0.0 0.0 0.0 " />
-	      <geometry name="l_index0__collision">
+	      <geometry name="index0_collision_left">
 		      <mesh filename="package://${MESH_COLL}/H2R3/H2R3_finger_knuckle1.stl" />
 	      </geometry>
       </collision>
     </link>
-    <joint name="left_hand_j4" type="revolute">
+    <joint name="left_hand_j5" type="revolute">
       <axis xyz="0 1 0" />
       <limit effort="100" velocity="${1600*M_PI/180}" lower="${-34.99*M_PI/180}" upper="${34.99*M_PI/180}" />
       <origin xyz="0 0 -0.044" rpy="0 0 0" />
-      <parent link="l_index0"/>
-      <child link="l_index1"/>
-    </joint>
-    <link name="l_index1">
+      <parent link="index0_left"/>
+      <child link="index1_left"/>
+    </joint>
+    <link name="index1_left">
       <inertial>
         <mass value="0.0429" />
@@ -186,5 +194,5 @@
 	      <material name="GreyC" />
 	      <origin xyz="0 0 0" rpy="0 0 0 " />
-	      <geometry name="l_index1_geom">
+	      <geometry name="index1_geom_left">
 		      <mesh filename="package://${MESH}/H2R3/H2R3_finger_knuckle2.dae" />
 	      </geometry>
@@ -192,31 +200,31 @@
       <collision>
 	      <origin xyz="0 0 0" rpy="0.0 0.0 0.0 " />
-	      <geometry name="l_index1_collision">
+	      <geometry name="index1_collision_left">
 		      <mesh filename="package://${MESH_COLL}/H2R3/H2R3_finger_knuckle2.stl" />
 	      </geometry>
       </collision>
     </link>
-    <joint name="left_hand_j5" type="revolute">
+    <joint name="left_hand_j6" type="revolute">
       <axis xyz="0 1 0" />
       <limit effort="100" velocity="${1600*M_PI/180}" lower="${-34.21*M_PI/180}" upper="${34.213*M_PI/180}" />
       <origin xyz="0 0 -0.032" rpy="0 0 0" />
-      <parent link="l_index1"/>
-      <child link="l_index2"/>
-    </joint>
-    <link name="l_index2">
-      <inertial>
-        <mass value="0.01" />
-	<origin xyz="0.0 0.0 0.0"/>
-	<inertia ixx="0.0"
-	iyy="0.0"
-	izz="0.0"
-	ixy="0.0"
-	ixz="0.0"
-	iyz="0.0" />
-      </inertial>
-      <visual>
-	      <material name="GreyC" />
-	      <origin xyz="0 0 0" rpy="0 0 0 " />
-	      <geometry name="l_index2_geom">
+      <parent link="index1_left"/>
+      <child link="index2_left"/>
+    </joint>
+    <link name="index2_left">
+      <inertial>
+        <mass value="0.01" />
+	<origin xyz="0.0 0.0 0.0"/>
+	<inertia ixx="0.0"
+	iyy="0.0"
+	izz="0.0"
+	ixy="0.0"
+	ixz="0.0"
+	iyz="0.0" />
+      </inertial>
+      <visual>
+	      <material name="GreyC" />
+	      <origin xyz="0 0 0" rpy="0 0 0 " />
+	      <geometry name="index2_geom_left">
 		      <mesh filename="package://${MESH}/H2R3/H2R3_finger_knuckle3.dae" />
 	      </geometry>
@@ -224,18 +232,26 @@
       <collision>
 	      <origin xyz="0 0 0" rpy="0.0 0.0 0.0 " />
-	      <geometry name="l_index2_collision">
+	      <geometry name="index2_collision_left">
 		      <mesh filename="package://${MESH_COLL}/H2R3/H2R3_finger_knuckle3.stl" />
 	      </geometry>
       </collision>
     </link>
+    <joint name="left_hand_j7" type="revolute">
+      <axis xyz="0 1 0" />
+      <limit effort="100" velocity="${1600*M_PI/180}" lower="${-34.21*M_PI/180}" upper="${34.213*M_PI/180}" />
+      <origin xyz="0 0.008 -0.025" rpy="0 0 0" />
+      <parent link="index2_left"/>
+      <child link="index_end_left"/>
+    </joint>
+    <link name="index_end_left"/>
 <!-- Start Ring Finger -->
-    <joint name="left_hand_j6" type="revolute">
+    <joint name="left_hand_j8" type="revolute">
       <axis xyz="0 1 0" />
       <origin xyz="0 0 -0.101" rpy="0 0 0" />
-      <parent link="l_palm" />
-      <child link="l_ring0"/>
+      <parent link="palm_left" />
+      <child link="ring0_left"/>
 	<limit effort="100" velocity="${50*M_PI/180}" lower="${-7.072*M_PI/180}" upper="${37.072*M_PI/180}" />
     </joint>
-    <link name="l_ring0">
+    <link name="ring0_left">
       <inertial>
         <mass value="0.01" />
@@ -251,5 +267,5 @@
 	      <material name="GreyA" />
 	      <origin xyz="0 0 0" rpy="0 0 0 " />
-	      <geometry name="l_ring0_geom">
+	      <geometry name="ring0_geom_left">
 		     <mesh filename="package://${MESH}/H2R3/H2R3_finger_knuckle1.dae" />
 	      </geometry>
@@ -257,17 +273,17 @@
       <collision>
 	      <origin xyz="0 0 0" rpy="0.0 0.0 0.0 " />
-	      <geometry name="l_ring0__collision">
+	      <geometry name="ring0_collision_left">
 		      <mesh filename="package://${MESH_COLL}/H2R3/H2R3_finger_knuckle1.stl" />
 	      </geometry>
       </collision>
     </link>
-    <joint name="left_hand_j7" type="revolute">
+    <joint name="left_hand_j9" type="revolute">
       <axis xyz="0 1 0" />
       <limit effort="100" velocity="${1600*M_PI/180}" lower="${-34.99*M_PI/180}" upper="${34.99*M_PI/180}" />
       <origin xyz="0 0 -0.044" rpy="0 0 0" />
-      <parent link="l_ring0"/>
-      <child link="l_ring1"/>
-    </joint>
-    <link name="l_ring1">
+      <parent link="ring0_left"/>
+      <child link="ring1_left"/>
+    </joint>
+    <link name="ring1_left">
       <inertial>
         <mass value="0.0429" />
@@ -283,5 +299,5 @@
 	      <material name="GreyC" />
 	      <origin xyz="0 0 0" rpy="0 0 0 " />
-	      <geometry name="l_ring1_geom">
+	      <geometry name="ring1_geom_left">
 		      <mesh filename="package://${MESH}/H2R3/H2R3_finger_knuckle2.dae" />
 	      </geometry>
@@ -289,31 +305,31 @@
       <collision>
 	      <origin xyz="0 0 0" rpy="0.0 0.0 0.0 " />
-	      <geometry name="l_ring1_collision">
+	      <geometry name="ring1_collision_left">
 		      <mesh filename="package://${MESH_COLL}/H2R3/H2R3_finger_knuckle2.stl" />
 	      </geometry>
       </collision>
     </link>
-    <joint name="left_hand_j8" type="revolute">
+    <joint name="left_hand_j10" type="revolute">
       <axis xyz="0 1 0" />
       <limit effort="100" velocity="${1600*M_PI/180}" lower="${-34.21*M_PI/180}" upper="${34.213*M_PI/180}" />
       <origin xyz="0 0 -0.032" rpy="0 0 0" />
-      <parent link="l_ring1"/>
-      <child link="l_ring2"/>
-    </joint>
-    <link name="l_ring2">
-      <inertial>
-        <mass value="0.01" />
-	<origin xyz="0.0 0.0 0.0"/>
-	<inertia ixx="0.0"
-	iyy="0.0"
-	izz="0.0"
-	ixy="0.0"
-	ixz="0.0"
-	iyz="0.0" />
-      </inertial>
-      <visual>
-	      <material name="GreyC" />
-	      <origin xyz="0 0 0" rpy="0 0 0 " />
-	      <geometry name="l_ring2_geom">
+      <parent link="ring1_left"/>
+      <child link="ring2_left"/>
+    </joint>
+    <link name="ring2_left">
+      <inertial>
+        <mass value="0.01" />
+	<origin xyz="0.0 0.0 0.0"/>
+	<inertia ixx="0.0"
+	iyy="0.0"
+	izz="0.0"
+	ixy="0.0"
+	ixz="0.0"
+	iyz="0.0" />
+      </inertial>
+      <visual>
+	      <material name="GreyC" />
+	      <origin xyz="0 0 0" rpy="0 0 0 " />
+	      <geometry name="ring2_geom_left">
 		      <mesh filename="package://${MESH}/H2R3/H2R3_finger_knuckle3.dae" />
 	      </geometry>
@@ -321,18 +337,26 @@
       <collision>
 	      <origin xyz="0 0 0" rpy="0.0 0.0 0.0 " />
-	      <geometry name="l_ring2_collision">
+	      <geometry name="ring2_collision_left">
 		      <mesh filename="package://${MESH_COLL}/H2R3/H2R3_finger_knuckle3.stl" />
 	      </geometry>
       </collision>
     </link>
+    <joint name="left_hand_j11" type="revolute">
+      <axis xyz="0 1 0" />
+      <limit effort="100" velocity="${1600*M_PI/180}" lower="${-34.21*M_PI/180}" upper="${34.213*M_PI/180}" />
+      <origin xyz="0 0.008 -0.025" rpy="0 0 0" />
+      <parent link="ring2_left"/>
+      <child link="ring_end_left"/>
+    </joint>
+    <link name="ring_end_left"/>
 <!-- Start Pinky Finger -->
-    <joint name="left_hand_j9" type="revolute">
+    <joint name="left_hand_j12" type="revolute">
       <axis xyz="0 1 0" />
       <origin xyz="0 -0.028 -0.101" rpy="0 0 0" />
-      <parent link="l_palm" />
-      <child link="l_pinky0"/>
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