Commit message: Added left arm/hand URDF

File: meka_description/urdf/H2R4_r_hand_defs.urdf.xacro (robot description, xacro)
@@ -5,10 +5,10 @@
   <property name="M_PI" value="3.1415926535897931" />
   <macro name="m3_r_palm" params="side parent reflect *origin">
-  <joint name="palm_joint" type="fixed">
+  <joint name="palm_joint_right" type="fixed">
     <origin xyz="0 0 -0.04414" rpy="0 0 0" />
     <parent link="${parent}"/>
-    <child link="palm" />
+    <child link="palm_right" />
   </joint>
-     <link name="palm">
+     <link name="palm_right">
       <inertial>
         <mass value="0.663" />
@@ -22,7 +22,7 @@
       </inertial>
       <visual>
-	      <material name="GreyA" />
-	      <origin xyz="0 0 0" rpy="0 0 0 " />
-	      <geometry name="palm_geom">
+	      <material name="GreyC" />
+	      <origin xyz="0 0 0" rpy="0 0 0 " />
+	      <geometry name="palm_geom_right">
 		      <mesh filename="package://${MESH}/H2R3/H2R3_RT8_palm_right.dae" />
 	      </geometry>
@@ -30,5 +30,5 @@
       <collision>
 	      <origin xyz="0 0 0" rpy="0.0 0.0 0.0 " />
-	      <geometry name="palm_collision">
+	      <geometry name="palm_collision_right">
 		      <mesh filename="package://${MESH_COLL}/H2R3/H2R3_RT8_palm_right.stl" />
 	      </geometry>
@@ -39,9 +39,9 @@
       <axis xyz="0 0 -1" />
       <origin xyz="-0.02 0.028 -0.03" rpy="0 0 0" />
-      <parent link="palm"/>
-      <child link="thumb0"/>
+      <parent link="palm_right"/>
+      <child link="thumb0_right"/>
       <limit effort="100" velocity="${20.0*M_PI/180}" lower="${-40*M_PI/180}" upper="${15*M_PI/180}" />
     </joint>
-    <link name="thumb0">
+    <link name="thumb0_right">
       <inertial>
         <mass value="0.0117" />
@@ -57,5 +57,5 @@
 	      <material name="GreyA" />
 	      <origin xyz="0 0 0" rpy="0 0 0 " />
-	      <geometry name="thumb0_geom">
+	      <geometry name="thumb0_geom_right">
 		      <mesh filename="package://${MESH}/H2R3/H2R3_RJ0_thumb_abductlink.dae" />
 	      </geometry>
@@ -63,5 +63,5 @@
       <collision>
 	      <origin xyz="0 0 0" rpy="0.0 0.0 0.0 " />
-	      <geometry name="thumb0_collision">
+	      <geometry name="thumb0_collision_right">
 		      <mesh filename="package://${MESH_COLL}/H2R3/H2R3_RJ0_thumb_abductlink.stl" />
 	      </geometry>
@@ -72,8 +72,8 @@
      <limit effort="100" velocity="${75*M_PI/180}" lower="${-80.919*M_PI/180}" upper="${80.91*M_PI/180}" />
       <origin xyz="-0.018 0 0" rpy="0 0 0" />
-      <parent link="thumb0"/>
-      <child link="thumb1"/>
-    </joint>
-    <link name="thumb1">
+      <parent link="thumb0_right"/>
+      <child link="thumb1_right"/>
+    </joint>
+    <link name="thumb1_right">
       <inertial>
         <mass value="0.0344" />
@@ -89,11 +89,11 @@
 	      <material name="GreyB" />
 	      <origin xyz="0 0 0" rpy="0 0 0 " />
-	      <geometry name="thumb1_geom">
-		      <mesh filename="package://${MESH}/H2R3/H2R3_thumb_knuckle1.dae" />
-	      </geometry>
-      </visual>
-      <collision>
-	      <origin xyz="0 0 0" rpy="0.0 0.0 0.0 " />
-	      <geometry name="thumb1_collision">
+	      <geometry name="thumb1_geom_right">
+		      <mesh filename="package://${MESH}/H2R3/H2R3_thumb_knuckle1.stl" />
+	      </geometry>
+      </visual>
+      <collision>
+	      <origin xyz="0 0 0" rpy="0.0 0.0 0.0 " />
+	      <geometry name="thumb1_collision_right">
 		      <mesh filename="package://${MESH_COLL}/H2R3/H2R3_thumb_knuckle1.stl" />
 	      </geometry>
@@ -103,23 +103,23 @@
       <axis xyz="0 -1 0" />
       <origin xyz="-0.044 0 0" rpy="0 0 0" />
-      <parent link="thumb1" />
-      <child link="thumb2"/>
+      <parent link="thumb1_right" />
+      <child link="thumb2_right"/>
       <limit effort="100" velocity="${50*M_PI/180}" lower="${-14.94*M_PI/180}" upper="${14.94*M_PI/180}" />
     </joint>
-    <link name="thumb2">
-      <inertial>
-        <mass value="0.01" />
-	<origin xyz="0.0 0.0 0.0"/>
-	<inertia ixx="0.0"
-	iyy="0.0"
-	izz="0.0"
-	ixy="0.0"
-	ixz="0.0"
-	iyz="0.0" />
-      </inertial>
-      <visual>
-	      <material name="GreyC" />
-	      <origin xyz="0 0 0" rpy="0 0 0 " />
-	      <geometry name="thumb_knuckle2_geom">
+    <link name="thumb2_right">
+      <inertial>
+        <mass value="0.01" />
+	<origin xyz="0.0 0.0 0.0"/>
+	<inertia ixx="0.0"
+	iyy="0.0"
+	izz="0.0"
+	ixy="0.0"
+	ixz="0.0"
+	iyz="0.0" />
+      </inertial>
+      <visual>
+	      <material name="GreyC" />
+	      <origin xyz="0 0 0" rpy="0 0 0 " />
+	      <geometry name="thumb_knuckle2_geom_right">
 		      <mesh filename="package://${MESH}/H2R3/H2R3_thumb_knuckle2.dae" />
 	      </geometry>
@@ -127,5 +127,5 @@
       <collision>
 	      <origin xyz="0 0 0" rpy="0.0 0.0 0.0 " />
-	      <geometry name="thumb_knuckle2_collision">
+	      <geometry name="thumb_knuckle2_collision_right">
 		      <mesh filename="package://${MESH_COLL}/H2R3/H2R3_thumb_knuckle2.stl" />
 	      </geometry>
@@ -135,18 +135,18 @@
       <axis xyz="0 -1 0" />
       <origin xyz="-0.035 0 0" rpy="0 0 0" />
-      <parent link="thumb2" />
-      <child link="thumb_end"/>
+      <parent link="thumb2_right" />
+      <child link="thumb_end_right"/>
       <limit effort="100" velocity="${50*M_PI/180}" lower="${-14.94*M_PI/180}" upper="${14.94*M_PI/180}" />
     </joint>
-    <link name="thumb_end"/>
+    <link name="thumb_end_right"/>
 <!-- Start Index Finger -->
     <joint name="right_hand_j4" type="revolute">
       <axis xyz="0 1 0" />
       <origin xyz="0 0.028 -0.101" rpy="0 0 0" />
-      <parent link="palm" />
-      <child link="index0"/>
+      <parent link="palm_right" />
+      <child link="index0_right"/>
 	<limit effort="100" velocity="${50*M_PI/180}" lower="${-7.072*M_PI/180}" upper="${37.072*M_PI/180}" />
     </joint>
-    <link name="index0">
+    <link name="index0_right">
       <inertial>
         <mass value="0.01" />
@@ -162,5 +162,5 @@
 	      <material name="GreyA" />
 	      <origin xyz="0 0 0" rpy="0 0 0 " />
-	      <geometry name="index0_geom">
+	      <geometry name="index0_geom_right">
 		     <mesh filename="package://${MESH}/H2R3/H2R3_finger_knuckle1.dae" />
 	      </geometry>
@@ -168,5 +168,5 @@
       <collision>
 	      <origin xyz="0 0 0" rpy="0.0 0.0 0.0 " />
-	      <geometry name="index0__collision">
+	      <geometry name="index0_collision_right">
 		      <mesh filename="package://${MESH_COLL}/H2R3/H2R3_finger_knuckle1.stl" />
 	      </geometry>
@@ -177,8 +177,8 @@
       <limit effort="100" velocity="${1600*M_PI/180}" lower="${-34.99*M_PI/180}" upper="${34.99*M_PI/180}" />
       <origin xyz="0 0 -0.044" rpy="0 0 0" />
-      <parent link="index0"/>
-      <child link="index1"/>
-    </joint>
-    <link name="index1">
+      <parent link="index0_right"/>
+      <child link="index1_right"/>
+    </joint>
+    <link name="index1_right">
       <inertial>
         <mass value="0.0429" />
@@ -194,5 +194,5 @@
 	      <material name="GreyC" />
 	      <origin xyz="0 0 0" rpy="0 0 0 " />
-	      <geometry name="index1_geom">
+	      <geometry name="index1_geom_right">
 		      <mesh filename="package://${MESH}/H2R3/H2R3_finger_knuckle2.dae" />
 	      </geometry>
@@ -200,5 +200,5 @@
       <collision>
 	      <origin xyz="0 0 0" rpy="0.0 0.0 0.0 " />
-	      <geometry name="index1_collision">
+	      <geometry name="index1_collision_right">
 		      <mesh filename="package://${MESH_COLL}/H2R3/H2R3_finger_knuckle2.stl" />
 	      </geometry>
@@ -209,22 +209,22 @@
       <limit effort="100" velocity="${1600*M_PI/180}" lower="${-34.21*M_PI/180}" upper="${34.213*M_PI/180}" />
       <origin xyz="0 0 -0.032" rpy="0 0 0" />
-      <parent link="index1"/>
-      <child link="index2"/>
-    </joint>
-    <link name="index2">
-      <inertial>
-        <mass value="0.01" />
-	<origin xyz="0.0 0.0 0.0"/>
-	<inertia ixx="0.0"
-	iyy="0.0"
-	izz="0.0"
-	ixy="0.0"
-	ixz="0.0"
-	iyz="0.0" />
-      </inertial>
-      <visual>
-	      <material name="GreyC" />
-	      <origin xyz="0 0 0" rpy="0 0 0 " />
-	      <geometry name="index2_geom">
+      <parent link="index1_right"/>
+      <child link="index2_right"/>
+    </joint>
+    <link name="index2_right">
+      <inertial>
+        <mass value="0.01" />
+	<origin xyz="0.0 0.0 0.0"/>
+	<inertia ixx="0.0"
+	iyy="0.0"
+	izz="0.0"
+	ixy="0.0"
+	ixz="0.0"
+	iyz="0.0" />
+      </inertial>
+      <visual>
+	      <material name="GreyC" />
+	      <origin xyz="0 0 0" rpy="0 0 0 " />
+	      <geometry name="index2_geom_right">
 		      <mesh filename="package://${MESH}/H2R3/H2R3_finger_knuckle3.dae" />
 	      </geometry>
@@ -232,5 +232,5 @@
       <collision>
 	      <origin xyz="0 0 0" rpy="0.0 0.0 0.0 " />
-	      <geometry name="index2_collision">
+	      <geometry name="index2_collision_right">
 		      <mesh filename="package://${MESH_COLL}/H2R3/H2R3_finger_knuckle3.stl" />
 	      </geometry>
@@ -241,17 +241,17 @@
       <limit effort="100" velocity="${1600*M_PI/180}" lower="${-34.21*M_PI/180}" upper="${34.213*M_PI/180}" />
       <origin xyz="0 0.008 -0.025" rpy="0 0 0" />
-      <parent link="index2"/>
-      <child link="index_end"/>
-    </joint>
-    <link name="index_end"/>
+      <parent link="index2_right"/>
+      <child link="index_end_right"/>
+    </joint>
+    <link name="index_end_right"/>
 <!-- Start Ring Finger -->
     <joint name="right_hand_j8" type="revolute">
       <axis xyz="0 1 0" />
       <origin xyz="0 0 -0.101" rpy="0 0 0" />
-      <parent link="palm" />
-      <child link="ring0"/>
+      <parent link="palm_right" />
+      <child link="ring0_right"/>
 	<limit effort="100" velocity="${50*M_PI/180}" lower="${-7.072*M_PI/180}" upper="${37.072*M_PI/180}" />
     </joint>
-    <link name="ring0">
+    <link name="ring0_right">
       <inertial>
         <mass value="0.01" />
@@ -267,5 +267,5 @@
 	      <material name="GreyA" />
 	      <origin xyz="0 0 0" rpy="0 0 0 " />
-	      <geometry name="ring0_geom">
+	      <geometry name="ring0_geom_right">
 		     <mesh filename="package://${MESH}/H2R3/H2R3_finger_knuckle1.dae" />
 	      </geometry>
@@ -273,5 +273,5 @@
       <collision>
 	      <origin xyz="0 0 0" rpy="0.0 0.0 0.0 " />
-	      <geometry name="ring0__collision">
+	      <geometry name="ring0_collision_right">
 		      <mesh filename="package://${MESH_COLL}/H2R3/H2R3_finger_knuckle1.stl" />
 	      </geometry>
@@ -282,8 +282,8 @@
       <limit effort="100" velocity="${1600*M_PI/180}" lower="${-34.99*M_PI/180}" upper="${34.99*M_PI/180}" />
       <origin xyz="0 0 -0.044" rpy="0 0 0" />
-      <parent link="ring0"/>
-      <child link="ring1"/>
-    </joint>
-    <link name="ring1">
+      <parent link="ring0_right"/>
+      <child link="ring1_right"/>
+    </joint>
+    <link name="ring1_right">
       <inertial>
         <mass value="0.0429" />
@@ -299,5 +299,5 @@
 	      <material name="GreyC" />
 	      <origin xyz="0 0 0" rpy="0 0 0 " />
-	      <geometry name="ring1_geom">
+	      <geometry name="ring1_geom_right">
 		      <mesh filename="package://${MESH}/H2R3/H2R3_finger_knuckle2.dae" />
 	      </geometry>
@@ -305,5 +305,5 @@
       <collision>
 	      <origin xyz="0 0 0" rpy="0.0 0.0 0.0 " />
-	      <geometry name="ring1_collision">
+	      <geometry name="ring1_collision_right">
 		      <mesh filename="package://${MESH_COLL}/H2R3/H2R3_finger_knuckle2.stl" />
 	      </geometry>
@@ -314,22 +314,22 @@
       <limit effort="100" velocity="${1600*M_PI/180}" lower="${-34.21*M_PI/180}" upper="${34.213*M_PI/180}" />
       <origin xyz="0 0 -0.032" rpy="0 0 0" />
-      <parent link="ring1"/>
-      <child link="ring2"/>
-    </joint>
-    <link name="ring2">
-      <inertial>
-        <mass value="0.01" />
-	<origin xyz="0.0 0.0 0.0"/>
-	<inertia ixx="0.0"
-	iyy="0.0"
-	izz="0.0"
-	ixy="0.0"
-	ixz="0.0"
-	iyz="0.0" />
-      </inertial>
-      <visual>
-	      <material name="GreyC" />
-	      <origin xyz="0 0 0" rpy="0 0 0 " />
-	      <geometry name="ring2_geom">
+      <parent link="ring1_right"/>
+      <child link="ring2_right"/>
+    </joint>
+    <link name="ring2_right">
+      <inertial>
+        <mass value="0.01" />
+	<origin xyz="0.0 0.0 0.0"/>
+	<inertia ixx="0.0"
+	iyy="0.0"
+	izz="0.0"
+	ixy="0.0"
+	ixz="0.0"
+	iyz="0.0" />
+      </inertial>
+      <visual>
+	      <material name="GreyC" />
+	      <origin xyz="0 0 0" rpy="0 0 0 " />
+	      <geometry name="ring2_geom_right">
 		      <mesh filename="package://${MESH}/H2R3/H2R3_finger_knuckle3.dae" />
 	      </geometry>
@@ -337,5 +337,5 @@
       <collision>
 	      <origin xyz="0 0 0" rpy="0.0 0.0 0.0 " />
-	      <geometry name="ring2_collision">
+	      <geometry name="ring2_collision_right">
 		      <mesh filename="package://${MESH_COLL}/H2R3/H2R3_finger_knuckle3.stl" />
 	      </geometry>
@@ -346,17 +346,17 @@
       <limit effort="100" velocity="${1600*M_PI/180}" lower="${-34.21*M_PI/180}" upper="${34.213*M_PI/180}" />
       <origin xyz="0 0.008 -0.025" rpy="0 0 0" />
-      <parent link="ring2"/>
-      <child link="ring_end"/>
-    </joint>
-    <link name="ring_end"/>
+      <parent link="ring2_right"/>
+      <child link="ring_end_right"/>
+    </joint>
+    <link name="ring_end_right"/>
 <!-- Start Pinky Finger -->
     <joint name="right_hand_j12" type="revolute">
       <axis xyz="0 1 0" />
       <origin xyz="0 -0.028 -0.101" rpy="0 0 0" />
-      <parent link="palm" />
-      <child link="pinky0"/>
+      <parent link="palm_right" />
+      <child link="pinky0_right"/>
 	<limit effort="100" velocity="${50*M_PI/180}" lower="${-7.072*M_PI/180}" upper="${37.072*M_PI/180}" />
     </joint>
-    <link name="pinky0">
+    <link name="pinky0_right">
       <inertial>
         <mass value="0.01" />
@@ -372,5 +372,5 @@
 	      <material name="GreyA" />
 	      <origin xyz="0 0 0" rpy="0 0 0 " />
-	      <geometry name="pinky0_geom">
+	      <geometry name="pinky0_geom_right">
 		     <mesh filename="package://${MESH}/H2R3/H2R3_finger_knuckle1.dae" />
 	      </geometry>
@@ -378,5 +378,5 @@
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
Commit message: fix full body URDF

File: meka_description/robots/ens.urdf.xacro (robot description, xacro)
@@ -15,5 +15,5 @@
  <!-- Solid Base -->
  <joint name="base_joint" type="fixed">
-  <origin xyz="0 0 1" rpy="0 0 0" />
+  <origin xyz="0 0 0" rpy="0 0 0" />
   <parent link="world" />
   <child link="base_link" />
@@ -40,4 +40,5 @@
   <!-- john added transmissions -->
   <xacro:include filename="$(find meka_description)/transmissions/A2R4_r_arm_defs.transmission.xacro" />
+  <xacro:include filename="$(find meka_description)/transmissions/A2R4_l_arm_defs.transmission.xacro" />
   <!--<xacro:include filename="$(find meka_description)/transmissions/H2R2_r_hand_defs.transmission.xacro" />-->
   <!--<xacro:include filename="$(find meka_description)/transmissions/S2R1_head_defs.transmission.xacro" />-->
@@ -53,8 +54,8 @@
   </material>
   <!-- john added transmissions -->
-  <xacro:m3_r_arm_transmission side="r" reflect="1" parent="upper"/>
-  <xacro:m3_l_arm_transmission side="r" reflect="1" parent="upper"/>
+  <xacro:m3_r_arm_transmission side="r" reflect="-1" parent="upper"/>
+  <xacro:m3_l_arm_transmission side="l" reflect="1" parent="upper"/>
   <!--</m3_r_hand_transmission-->
-  <xacro:m3_r_hand side="r" reflect="1" parent="handmount_RIGHT">
+  <xacro:m3_r_hand side="r" reflect="-1" parent="handmount_RIGHT">
     <origin xyz="0.0 0.0 0.0" rpy="0 0 0" />
   </xacro:m3_r_hand>
@@ -65,5 +66,5 @@
     <origin xyz="0.0 0.0 0.31155" rpy="0 0 0" />
   </xacro:m3_head>
- <xacro:m3_r_arm side="r" reflect="1" parent="upper">
+ <xacro:m3_r_arm side="r" reflect="-1" parent="upper">
     <origin xyz="0.0 -0.18465 0.2337" rpy="0 0 0" />
   </xacro:m3_r_arm>

File: meka_description/transmissions/A2R2_r_arm_defs.transmission.xacro (robot description, xacro)
@@ -3,5 +3,5 @@
        xmlns:controller="http://playerstage.sourceforge.net/gazebo/xmlschema/#controller"
        xmlns:interface="http://playerstage.sourceforge.net/gazebo/xmlschema/#interface">
-  <macro name="m3_r_shoulder_transmission" params="side parent reflect">
+  <xacro:macro name="m3_r_shoulder_transmission" params="side parent reflect">
     <!-- Shoulder pan -->
     <transmission name="m3joint_${R_ARM}_t0" type="pr2_mechanism_model/SimpleTransmission">
@@ -22,7 +22,7 @@
       <mechanicalReduction>1</mechanicalReduction>
     </transmission>
-  </macro>
+  </xacro:macro>
   <!-- ============================   Upper Arm   ============================ -->
-  <macro name="m3_r_upper_arm_transmission" params="side parent reflect">
+  <xacro:macro name="m3_r_upper_arm_transmission" params="side parent reflect">
     <transmission name="m3joint_${R_ARM}_t3" type="pr2_mechanism_model/SimpleTransmission">
       <actuator name="m3joint_${R_ARM}_a3" />
@@ -36,7 +36,7 @@
       <mechanicalReduction>1</mechanicalReduction>
     </transmission>
-  </macro>
+  </xacro:macro>
   <!-- ============================   Forearm   ============================ -->
-  <macro name="m3_r_forearm_transmission" params="side parent reflect">
+  <xacro:macro name="m3_r_forearm_transmission" params="side parent reflect">
     <transmission name="m3joint_${R_ARM}_t5" type="pr2_mechanism_model/SimpleTransmission">
       <actuator name="m3joint_${R_ARM}_a5" />
@@ -50,9 +50,9 @@
       <mechanicalReduction>1</mechanicalReduction>
     </transmission>
-  </macro>
-  <macro name="m3_r_arm_transmission" params="side parent reflect">
+  </xacro:macro>
+  <xacro:macro name="m3_r_arm_transmission" params="side parent reflect">
     <m3_r_shoulder_transmission side="${side}" reflect="${reflect}" parent="${parent}"/>
     <m3_r_upper_arm_transmission side="${side}" reflect="${reflect}" parent="bicep_RIGHT" />
     <m3_r_forearm_transmission side="${side}" reflect="${reflect}" parent="wrist_RIGHT" />
-  </macro>
+  </xacro:macro>
 </robot>

File: meka_description/transmissions/A2R3_l_arm_defs.transmission.xacro (robot description, xacro)
@@ -3,5 +3,5 @@
        xmlns:controller="http://playerstage.sourceforge.net/gazebo/xmlschema/#controller"
        xmlns:interface="http://playerstage.sourceforge.net/gazebo/xmlschema/#interface">
-  <macro name="m3_l_shoulder_transmission" params="side parent reflect *origin">
+  <xacro:macro name="m3_l_shoulder_transmission" params="side parent reflect *origin">
     <!-- Shoulder pan -->
     <transmission name="m3joint_${L_ARM}_t0" type="pr2_mechanism_model/SimpleTransmission">
@@ -22,7 +22,7 @@
       <mechanicalReduction>1</mechanicalReduction>
     </transmission>
-  </macro>
+  </xacro:macro>
   <!-- ============================   Upper Arm   ============================ -->
-  <macro name="m3_l_upper_arm_transmission" params="side parent reflect">
+  <xacro:macro name="m3_l_upper_arm_transmission" params="side parent reflect">
     <transmission name="m3joint_${L_ARM}_t3" type="pr2_mechanism_model/SimpleTransmission">
       <actuator name="m3joint_${L_ARM}_a3" />
@@ -36,7 +36,7 @@
       <mechanicalReduction>1</mechanicalReduction>
     </transmission>
-  </macro>
+  </xacro:macro>
   <!-- ============================   Forearm   ============================ -->
-  <macro name="m3_l_forearm_transmission" params="side parent reflect">
+  <xacro:macro name="m3_l_forearm_transmission" params="side parent reflect">
     <transmission name="m3joint_${L_ARM}_t5" type="pr2_mechanism_model/SimpleTransmission">
       <actuator name="m3joint_${L_ARM}_a5" />
@@ -50,9 +50,9 @@
       <mechanicalReduction>1</mechanicalReduction>
     </transmission>
-  </macro>
-  <macro name="m3_l_arm_transmission" params="side parent reflect *origin">
+  </xacro:macro>
+  <xacro:macro name="m3_l_arm_transmission" params="side parent reflect *origin">
     <m3_l_shoulde_transmissionr side="${side}" reflect="${reflect}" parent="${parent}"/>
     <m3_l_upper_ar_transmissionm side="${side}" reflect="${reflect}" parent="bicep_LEFT" />
     <m3_l_forear_transmissionm side="${side}" reflect="${reflect}" parent="wrist_LEFT" />
-  </macro>
+  </xacro:macro>
 </robot>

File: meka_description/urdf/H2R4_l_hand_defs.urdf.xacro (robot description, xacro)
@@ -31,5 +31,5 @@
 	      <origin xyz="0 0 0" rpy="0.0 0.0 0.0 " />
 	      <geometry name="palm_collision_left">
-		      <mesh filename="package://${MESH_COLL}/H2R3/H2R3_LT8_palm_left.dae" />
+		      <mesh filename="package://${MESH_COLL}/H2R3/H2R3_LT8_palm_left.stl" />
 	      </geometry>
       </collision>

Commit message: removed gazebo

File: meka_description/robots/ens.urdf.xacro (robot description, xacro)
@@ -8,6 +8,6 @@
  <property name="MESH" value="meka_description/meshes/mid_res" />
  <property name="MESH_COLL" value="meka_description/meshes/low_res" />
-<!-- generic simulator_gazebo plugins for starting mechanism control, ros time, ros battery -->
- <xacro:include filename="$(find meka_description)/gazebo/gazebo.urdf.xacro" />
+<!-- generic simulator_gazebo plugins for starting mechanism control, ros time, ros battery >
+ <xacro:include filename="$(find meka_description)/gazebo/gazebo.urdf.xacro" /-->
  <!--<xacro:include filename="$(find meka_description)/transmissions/uta.transmission.xacro" />-->
  <link name="world" />
@@ -38,7 +38,7 @@
 <!-- Meka Head -->
   <xacro:include filename="$(find meka_description)/urdf/ENS_head_defs.urdf.xacro" />
-  <!-- john added transmissions -->
+  <!-- john added transmissions >
   <xacro:include filename="$(find meka_description)/transmissions/A2R4_r_arm_defs.transmission.xacro" />
-  <xacro:include filename="$(find meka_description)/transmissions/A2R4_l_arm_defs.transmission.xacro" />
+  <xacro:include filename="$(find meka_description)/transmissions/A2R4_l_arm_defs.transmission.xacro" /-->
   <!--<xacro:include filename="$(find meka_description)/transmissions/H2R2_r_hand_defs.transmission.xacro" />-->
   <!--<xacro:include filename="$(find meka_description)/transmissions/S2R1_head_defs.transmission.xacro" />-->
@@ -53,7 +53,7 @@
     <color rgba="0.7 0.7 0.7 1.0"/>
   </material>
-  <!-- john added transmissions -->
+  <!-- john added transmissions >
   <xacro:m3_r_arm_transmission side="r" reflect="-1" parent="upper"/>
-  <xacro:m3_l_arm_transmission side="l" reflect="1" parent="upper"/>
+  <xacro:m3_l_arm_transmission side="l" reflect="1" parent="upper"/-->
   <!--</m3_r_hand_transmission-->
   <xacro:m3_r_hand side="r" reflect="-1" parent="handmount_RIGHT">

File: meka_description/urdf/A2R4_l_arm_defs.urdf.xacro (robot description, xacro)
@@ -130,5 +130,4 @@
       <child link="elbowclevis_LEFT"/>
 	<limit effort="20" velocity="${50*M_PI/180}" lower="${-0.278978*M_PI/180}" upper="${132.8175*M_PI/180}" />
-      <dynamics damping="10.0" />
     </joint>
     <link name="elbowclevis_LEFT">
